Commit message: albatross lives in sim

File: tauv_config/albatross_description/urdf/actuators.xacro (robot description, xacro)
@@ -8,25 +8,43 @@
           aware that Gazebo does not use the SNAME convention per default.
     -->
-    <xacro:thruster_macro robot_namespace="${namespace}" thruster_id="0">
-        <origin xyz="0 0 0" rpy="0 0 ${pi}" />
-    </xacro:thruster_macro>
-    <xacro:thruster_macro robot_namespace="${namespace}" thruster_id="1">
-        <origin xyz="0 0 0" rpy="0 0 ${pi}" />
-    </xacro:thruster_macro>
-    <xacro:thruster_macro robot_namespace="${namespace}" thruster_id="2">
-    <origin xyz="0 0 0" rpy="0 -${0.5*pi} 0" />
-    </xacro:thruster_macro>
-    <!-- Instantiate fins, if necessary -->
-    <xacro:fin_macro namespace="${namespace}" fin_id="0">
-      <origin xyz="0 0 0" rpy="0 0 0" />
-    </xacro:fin_macro>
-    <xacro:fin_macro namespace="${namespace}" fin_id="1">
-      <origin xyz="0 0 0" rpy="0 0 0" />
-    </xacro:fin_macro>
-    <xacro:fin_macro namespace="${namespace}" fin_id="2">
-      <origin xyz="0 0 0" rpy="0 0 0" />
-    </xacro:fin_macro>
-    <xacro:fin_macro namespace="${namespace}" fin_id="3">
-      <origin xyz="0 0 0" rpy="0 0 0" />
-    </xacro:fin_macro>
+  <xacro:property name="prop_mesh_file_cw" value="file://$(find albatross_description)/meshes/t200_propccw.dae"/>
+  <xacro:property name="prop_mesh_file_ccw" value="file://$(find albatross_description)/meshes/t200_propcw.dae"/>
+  <xacro:macro name="thruster_macro"
+    params="namespace thruster_id *origin">
+    <xacro:thruster_module_first_order_basic_fcn_macro
+      namespace="${namespace}"
+      thruster_id="${thruster_id}"
+      mesh_filename="${prop_mesh_file_cw}"
+      dyn_time_constant="0.2"
+      rotor_constant="0.000004">
+      <xacro:insert_block name="origin"/>
+    </xacro:thruster_module_first_order_basic_fcn_macro>
+  </xacro:macro>
+<!-- Top thrusters -->
+  <xacro:thruster_macro namespace="${namespace}" thruster_id="0"> <!-- heave back left prop up-->
+  <origin xyz="-0.12070 0.12070 0" rpy="0 -1.5707963268 0"/>
+  </xacro:thruster_macro>
+  <xacro:thruster_macro namespace="${namespace}" thruster_id="1"> <!-- heave bacl right prop up-->
+    <origin xyz="-0.12070 -0.12070 0" rpy="0 -1.5707963268 0"/>
+  </xacro:thruster_macro>
+  <xacro:thruster_macro namespace="${namespace}" thruster_id="2"> <!-- heave front left prop up-->
+    <origin xyz="0.12070 0.12070 0" rpy="0 -1.5707963268 0"/>
+  </xacro:thruster_macro>
+  <xacro:thruster_macro namespace="${namespace}" thruster_id="3"> <!-- heave front right prop up-->
+    <origin xyz="0.12070 -0.12070 0" rpy="0 -1.5707963268 0"/>
+  </xacro:thruster_macro>
+ <!-- Front thrusters -->
+  <xacro:thruster_macro namespace="${namespace}" thruster_id="6"> <!-- lat front left-->
+    <origin xyz="0.20506 0.20506 0" rpy="${0*d2r} ${0*d2r} ${135*d2r}"/>
+  </xacro:thruster_macro>
+  <xacro:thruster_macro namespace="${namespace}" thruster_id="7"> <!-- lat front right -->
+    <origin xyz="0.20506 -0.20506 0" rpy="${0*d2r} ${0*d2r} ${-135*d2r}"/>
+  </xacro:thruster_macro>
+ <!-- Back thrusters -->
+  <xacro:thruster_macro namespace="${namespace}" thruster_id="4"> <!-- lat back left-->
+    <origin xyz="-0.20506 0.20506 0" rpy="${0*d2r} ${0*d2r} ${45*d2r}"/>
+  </xacro:thruster_macro>
+  <xacro:thruster_macro namespace="${namespace}" thruster_id="5"> <!-- lat back right -->
+    <origin xyz="-0.20506 -0.20506 0" rpy="${0*d2r} ${0*d2r} ${-45*d2r}"/>
+  </xacro:thruster_macro>
 </robot>

File: tauv_config/albatross_description/urdf/base.xacro (robot description, xacro)
@@ -12,5 +12,5 @@
     Vehicle's parameters (remember to enter the model parameters below)
   -->
-  <xacro:property name="mass" value="0"/>
+  <xacro:property name="mass" value="15"/>
   <!-- Center of gravity -->
   <xacro:property name="cog" value="0 0 0"/>
@@ -39,7 +39,7 @@
           <mass value="${mass}" />
           <origin xyz="${cog}" rpy="0 0 0"/>
-          <inertia ixx="0" ixy="0" ixz="0"
-                   iyy="0" iyz="0"
-                   izz="0" />
+          <inertia
+            ixx="${0.503217}" ixy="${0.000204}" ixz="${-0.000526}"
+            iyy="${0.493449}" iyz="${0.000038}" izz="${0.919819}" />
         </inertial>
         <visual>

File: tauv_config/albatross_description/urdf/gazebo.xacro (robot description, xacro)
@@ -4,9 +4,9 @@
     <xacro:property name="albatross_cob" value="0 0 0"/>
     <!-- Vehicle's actual volume (Gazebo cannot compute the volume out of the mesh) -->
-    <xacro:property name="albatross_volume" value="0"/>
+    <xacro:property name="albatross_volume" value="0.01854"/>
     <!-- Describing the dimensions of the vehicle's bounding box -->
-    <xacro:property name="albatross_length" value="0"/>
-    <xacro:property name="albatross_width"  value="0"/>
-    <xacro:property name="albatross_height" value="0"/>
+    <xacro:property name="albatross_length" value="1"/>
+    <xacro:property name="albatross_width"  value="1"/>
+    <xacro:property name="albatross_height" value="1"/>
     <xacro:macro name="albatross_hydro_model" params="namespace">
       <!-- List of hydrodynamic models this robot's links -->
@@ -35,55 +35,58 @@
         <!-- 1) Fossen's equation of motion -->
         <hydrodynamic_model>
-          <type>fossen</type>
-          <added_mass>
-            0 0 0 0 0 0
-            0 0 0 0 0 0
-            0 0 0 0 0 0
-            0 0 0 0 0 0
-            0 0 0 0 0 0
-            0 0 0 0 0 0
-          </added_mass>
-          <!--
-            The linear damping coefficients can be provided as a diagonal (6 elements)
-            or a full matrix (36 coefficients), like the added-mass coefficients above
-          -->
-          <linear_damping>
-            0 0 0 0 0 0
-          </linear_damping>
-          <!--
-            The linear damping coefficients proportional to the forward speed
-            can be provided as a diagonal (6 elements) or a full matrix (36 coefficients),
-            like the added-mass coefficients above.
-            This matrix is mostly useful for slender bodies (e.g. AUVs with torpedo shape)
-          -->
-          <linear_damping_forward_speed>
-            0 0 0 0 0 0
-          </linear_damping_forward_speed>
-          <!--
-            The quadratic damping coefficients can be provided as a diagonal (6 elements)
-            or a full matrix (36 coefficients), like the added-mass coefficients above
-          -->
-          <quadratic_damping>
-            0 0 0 0 0 0
-          </quadratic_damping>
-          <!--
-            In case you want to model a simple surface vessel, you can use the
-            implementation of linear (small angle) theory for boxed shaped vessels
-            by providing the following parameters. If you omit the area of the
-            water level plane area, it will be calculated from the bounding box
-            parameters. Uncomment the lines below in case you are simulating a
-            surface vessel.
-            For more details on these parameters and the computation of buoyancy
-            for vessels using this theory, check:
-              [1] Lecture Notes  TTK 4190 Guidance and Control of Vehicles (T. I. Fossen)
-                  http://www.fossen.biz/wiley/Ch4.pdf
-              [2] Fossen, Thor I. Handbook of marine craft hydrodynamics and motion
-                  control. John Wiley & Sons, 2011.
-          -->
-          <!--
-          <metacentric_width>0.0</metacentric_width>
-          <metacentric_length>0.0</metacentric_length>
-          <submerged_height>0.0</submerged_height>
-          -->
+            <type>fossen</type>
+            <!-- Added mass: see p.28 in Berg2012 -->
+            <added_mass>
+              10.7727 0 0 0 0 0
+              0 10.7727 0 0 0 0
+              0 0 49.7679 0 0 0
+              0 0 0 1.0092 0 0
+              0 0 0 0 1.0092 0
+              0  0  0  0  0  0
+            </added_mass>
+            <!--
+              The linear damping coefficients can be provided as a diagonal (6 elements)
+              or a full matrix (36 coefficients), like the added-mass coefficients above
+              Linear damping: see p.31 in Berg2012
+            -->
+            <linear_damping>
+              -9.5909 -9.5909 -42.5798 -13.3040 -13.2181 -1.1559
+            </linear_damping>
+            <!--
+              The linear damping coefficients proportional to the forward speed
+              can be provided as a diagonal (6 elements) or a full matrix (36 coefficients),
+              like the added-mass coefficients above.
+              This matrix is mostly useful for slender bodies (e.g. AUVs with torpedo shape)
+            -->
+            <!-- <linear_damping_forward_speed>
+              0 0 0 0 0 0
+            </linear_damping_forward_speed> -->
+            <!--
+              The quadratic damping coefficients can be provided as a diagonal (6 elements)
+              or a full matrix (36 coefficients), like the added-mass coefficients above
+              Non-linear damping: see p.30 in Berg2012
+            -->
+            <quadratic_damping>
+              -5.1386 -5.1386 -26.1105 0 0 0
+            </quadratic_damping>
+            <!--
+              In case you want to model a simple surface vessel, you can use the
+              implementation of linear (small angle) theory for boxed shaped vessels
+              by providing the following parameters. If you omit the area of the
+              water level plane area, it will be calculated from the bounding box
+              parameters. Uncomment the lines below in case you are simulating a
+              surface vessel.
+              For more details on these parameters and the computation of buoyancy
+              for vessels using this theory, check:
+                [1] Lecture Notes  TTK 4190 Guidance and Control of Vehicles (T. I. Fossen)
+                    http://www.fossen.biz/wiley/Ch4.pdf
+                [2] Fossen, Thor I. Handbook of marine craft hydrodynamics and motion
+                    control. John Wiley & Sons, 2011.
+            -->
+            <!--
+            <metacentric_width>0.0</metacentric_width>
+            <metacentric_length>0.0</metacentric_length>
+            <water_level_plane_area>0.0</water_level_plane_area>
+            -->
         </hydrodynamic_model>
         <!-- 2) This computes the added-mass and damping parameters for a sphere

Commit message: remap thruster numberings

File: tauv_config/albatross_description/urdf/actuators.xacro (robot description, xacro)
@@ -21,30 +21,32 @@
     </xacro:thruster_module_first_order_basic_fcn_macro>
   </xacro:macro>
-<!-- Top thrusters -->
-  <xacro:thruster_macro namespace="${namespace}" thruster_id="0"> <!-- heave back left prop up-->
-  <origin xyz="-0.12070 0.12070 0" rpy="0 -1.5707963268 0"/>
+  <!-- Top thrusters -->
+  <xacro:thruster_macro namespace="${namespace}" thruster_id="7"> <!-- heave back left prop down-->
+  <origin xyz="-0.12070 0.12070 0" rpy="0 1.5707963268 0"/>
   </xacro:thruster_macro>
-  <xacro:thruster_macro namespace="${namespace}" thruster_id="1"> <!-- heave bacl right prop up-->
-    <origin xyz="-0.12070 -0.12070 0" rpy="0 -1.5707963268 0"/>
+  <xacro:thruster_macro namespace="${namespace}" thruster_id="6"> <!-- heave bacl right prop down-->
+    <origin xyz="-0.12070 -0.12070 0" rpy="0 1.5707963268 0"/>
   </xacro:thruster_macro>
-  <xacro:thruster_macro namespace="${namespace}" thruster_id="2"> <!-- heave front left prop up-->
-    <origin xyz="0.12070 0.12070 0" rpy="0 -1.5707963268 0"/>
+  <xacro:thruster_macro namespace="${namespace}" thruster_id="5"> <!-- heave front left prop down-->
+    <origin xyz="0.12070 0.12070 0" rpy="0 1.5707963268 0"/>
   </xacro:thruster_macro>
-  <xacro:thruster_macro namespace="${namespace}" thruster_id="3"> <!-- heave front right prop up-->
-    <origin xyz="0.12070 -0.12070 0" rpy="0 -1.5707963268 0"/>
+  <xacro:thruster_macro namespace="${namespace}" thruster_id="4"> <!-- heave front right prop down-->
+    <origin xyz="0.12070 -0.12070 0" rpy="0 1.5707963268 0"/>
   </xacro:thruster_macro>
- <!-- Front thrusters -->
-  <xacro:thruster_macro namespace="${namespace}" thruster_id="6"> <!-- lat front left-->
-    <origin xyz="0.20506 0.20506 0" rpy="${0*d2r} ${0*d2r} ${135*d2r}"/>
+  <!-- Front thrusters -->
+  <xacro:thruster_macro namespace="${namespace}" thruster_id="1"> <!-- lat front left-->
+    <origin xyz="0.20506 0.20506 0" rpy="${0*d2r} ${0*d2r} ${-45*d2r}"/>
   </xacro:thruster_macro>
-  <xacro:thruster_macro namespace="${namespace}" thruster_id="7"> <!-- lat front right -->
-    <origin xyz="0.20506 -0.20506 0" rpy="${0*d2r} ${0*d2r} ${-135*d2r}"/>
+  <xacro:thruster_macro namespace="${namespace}" thruster_id="0"> <!-- lat front right -->
+    <origin xyz="0.20506 -0.20506 0" rpy="${0*d2r} ${0*d2r} ${45*d2r}"/>
   </xacro:thruster_macro>
- <!-- Back thrusters -->
-  <xacro:thruster_macro namespace="${namespace}" thruster_id="4"> <!-- lat back left-->
+  <!-- Back thrusters -->
+  <xacro:thruster_macro namespace="${namespace}" thruster_id="3"> <!-- lat back left-->
     <origin xyz="-0.20506 0.20506 0" rpy="${0*d2r} ${0*d2r} ${45*d2r}"/>
   </xacro:thruster_macro>
-  <xacro:thruster_macro namespace="${namespace}" thruster_id="5"> <!-- lat back right -->
+  <xacro:thruster_macro namespace="${namespace}" thruster_id="2"> <!-- lat back right -->
     <origin xyz="-0.20506 -0.20506 0" rpy="${0*d2r} ${0*d2r} ${-45*d2r}"/>
   </xacro:thruster_macro>
+  <!-- reminder: REP 103. x,y,z are forward, left, up. rpy are rotation about those axes -->
+  <!-- reminder: right hand rule: positive pitch is down, positive yaw is left, positive roll is right -->
 </robot>

Commit message: add thruster inversion array, update URDF

File: tauv_config/albatross_description/urdf/actuators.xacro (robot description, xacro)
@@ -43,8 +43,8 @@
   <!-- Back thrusters -->
   <xacro:thruster_macro namespace="${namespace}" thruster_id="3"> <!-- lat back left-->
-    <origin xyz="-0.20506 0.20506 0" rpy="${0*d2r} ${0*d2r} ${45*d2r}"/>
+    <origin xyz="-0.20506 0.20506 0" rpy="${0*d2r} ${0*d2r} ${-135*d2r}"/>
   </xacro:thruster_macro>
   <xacro:thruster_macro namespace="${namespace}" thruster_id="2"> <!-- lat back right -->
-    <origin xyz="-0.20506 -0.20506 0" rpy="${0*d2r} ${0*d2r} ${-45*d2r}"/>
+    <origin xyz="-0.20506 -0.20506 0" rpy="${0*d2r} ${0*d2r} ${135*d2r}"/>
   </xacro:thruster_macro>
   <!-- reminder: REP 103. x,y,z are forward, left, up. rpy are rotation about those axes -->
