Commit message: remove all known instances of tf prefixing

File: tauv_config/albatross_description/urdf/base.xacro (robot description, xacro)
@@ -31,5 +31,5 @@
   <xacro:macro name="albatross_base" params="namespace *gazebo">
       <!-- Rigid body description of the base link -->
-      <link name="${namespace}/base_link">
+      <link name="base_link">
         <!--
           Be careful to setup the coefficients for the inertial tensor,
@@ -56,5 +56,5 @@
         </collision>
       </link>
-    <gazebo reference="${namespace}/base_link">
+    <gazebo reference="base_link">
       <selfCollide>false</selfCollide>
     </gazebo>

File: tauv_config/albatross_description/urdf/gazebo.xacro (robot description, xacro)
@@ -11,5 +11,5 @@
     <xacro:macro name="albatross_hydro_model" params="namespace">
       <!-- List of hydrodynamic models this robot's links -->
-      <link name="${namespace}/base_link">
+      <link name="base_link">
         <!-- This flag will make the link neutrally buoyant -->
         <neutrally_buoyant>0</neutrally_buoyant>

File: tauv_config/albatross_description/urdf/sensors.xacro (robot description, xacro)
@@ -8,32 +8,32 @@
   -->
   <!-- Mount a GPS. -->
-  <xacro:default_gps namespace="${namespace}" parent_link="${namespace}/base_link" />
+  <xacro:default_gps namespace="${namespace}" parent_link="base_link" />
   <!-- Mount a Pose 3D sensor. -->
-  <xacro:default_pose_3d namespace="${namespace}" parent_link="${namespace}/base_link" />
+  <xacro:default_pose_3d namespace="${namespace}" parent_link="base_link" />
   <!-- Forward-looking sonar sensor -->
-  <xacro:forward_multibeam_p900 namespace="${namespace}" parent_link="${namespace}/base_link">
+  <xacro:forward_multibeam_p900 namespace="${namespace}" parent_link="base_link">
     <origin xyz="0 0 0" rpy="0 0 0"/>
   </xacro:forward_multibeam_p900>
   <!-- DVL  -->
-  <xacro:default_dvl namespace="${namespace}" parent_link="${namespace}/base_link">
+  <xacro:default_dvl namespace="${namespace}" parent_link="base_link">
     <origin xyz="0 0 0" rpy="0 0 0"/>
   </xacro:default_dvl>
   <!-- RPT  -->
-  <xacro:default_rpt namespace="${namespace}" parent_link="${namespace}/base_link">
+  <xacro:default_rpt namespace="${namespace}" parent_link="base_link">
     <origin xyz="0 0 0" rpy="0 0 0"/>
   </xacro:default_rpt>
   <!-- Pressure  -->
-  <xacro:default_pressure namespace="${namespace}" parent_link="${namespace}/base_link">
+  <xacro:default_pressure namespace="${namespace}" parent_link="base_link">
     <origin xyz="0 0 0" rpy="0 0 0"/>
   </xacro:default_pressure>
   <!-- IMU  -->
-  <xacro:default_imu namespace="${namespace}" parent_link="${namespace}/base_link">
+  <xacro:default_imu namespace="${namespace}" parent_link="base_link">
     <origin xyz="0 0 0" rpy="${0} ${90*d2r} ${-90*d2r}"/>
   </xacro:default_imu>
   <!-- Mount a camera -->
-  <xacro:default_camera namespace="${namespace}" parent_link="${namespace}/base_link" suffix="front">
+  <xacro:default_camera namespace="${namespace}" parent_link="base_link" suffix="front">
     <origin xyz="0.29 0.0 0." rpy="0 0 0"/>
   </xacro:default_camera>
-  <xacro:default_camera namespace="${namespace}" parent_link="${namespace}/base_link" suffix="under">
+  <xacro:default_camera namespace="${namespace}" parent_link="base_link" suffix="under">
     <origin xyz="0.15 0.0 -0.06" rpy="0 ${0.5*pi} 0"/>
   </xacro:default_camera>

File: tauv_config/albatross_description/urdf/snippets.xacro (robot description, xacro)
@@ -18,5 +18,5 @@
     of the vehicle and may cause internal collisions if set otherwise
     -->
-    <link name="${robot_namespace}/thruster_${thruster_id}">
+    <link name="thruster_${thruster_id}">
       <visual>
         <geometry>
@@ -36,6 +36,6 @@
       <xacro:insert_block name="origin" />
       <axis xyz="1 0 0" />
-      <parent link="${robot_namespace}/base_link" />
-      <child link="${robot_namespace}/thruster_${thruster_id}" />
+      <parent link="base_link" />
+      <child link="thruster_${thruster_id}" />
     </joint>
     <gazebo>
@@ -169,12 +169,12 @@
   <xacro:property name="fin_max_joint_limit" value="${0.0 * d2r}"/>
   <xacro:macro name="fin_macro" params="namespace fin_id *origin">
-      <joint name="${namespace}/fin${fin_id}_joint" type="revolute">
+      <joint name="fin${fin_id}_joint" type="revolute">
           <limit effort="0" lower="${fin_min_joint_limit}" upper="${fin_max_joint_limit}" velocity="0"/>
           <xacro:insert_block name="origin"/>
           <axis xyz="0 0 1"/>
-          <parent link="${namespace}/base_link" />
-          <child link="${namespace}/fin${fin_id}" />
+          <parent link="base_link" />
+          <child link="fin${fin_id}" />
       </joint>
-      <link name="${namespace}/fin${fin_id}">
+      <link name="fin${fin_id}">
         <inertial>
           <mass value="0.001" />
@@ -238,6 +238,6 @@
           <current_velocity_topic>/hydrodynamics/current_velocity</current_velocity_topic>
           <!-- Name of the correspodent fin link and joint  -->
-          <link_name>${namespace}/fin${fin_id}</link_name>
-          <joint_name>${namespace}/fin${fin_id}_joint</joint_name>
+          <link_name>in${fin_id}</link_name>
+          <joint_name>fin${fin_id}_joint</joint_name>
           <!-- Output topic to publish the current angle of the fin joint -->
           <output_topic>${namespace}/fins/${fin_id}/output</output_topic>

File: uuv-simulator/uuv_gazebo_plugins/uuv_gazebo_ros_plugins/urdf/battery_snippets.xacro (robot description, xacro)
@@ -14,5 +14,5 @@
             voltage
             update_rate">
-    <link name="${namespace}/battery_link">
+    <link name="battery_link">
       <inertial>
         <inertia ixx="0.00001" ixy="0.0" ixz="0.0" iyy="0.00001" iyz="0.0" izz="0.00001" />
@@ -21,13 +21,13 @@
       </inertial>
     </link>
-    <joint name="${namespace}/battery_joint" type="revolute">
+    <joint name="battery_joint" type="revolute">
       <origin xyz="0 0 0" rpy="0 0 0" />
       <parent link="${parent_link}" />
-      <child link="${namespace}/battery_link" />
+      <child link="battery_link" />
       <axis xyz="1 0 0"/>
       <limit upper="0" lower="0" effort="0" velocity="0" />
     </joint>
-    <gazebo reference="${namespace}/battery_link">
-      <battery name="${namespace}/battery">
+    <gazebo reference="battery_link">
+      <battery name="battery">
         <voltage>${voltage}</voltage>
       </battery>
@@ -37,6 +37,6 @@
         name="${namespace}_${prefix}linear_battery_ros_plugin">
         <namespace>${namespace}</namespace>
-        <link_name>${namespace}/battery_link</link_name>
-        <battery_name>${namespace}/battery</battery_name>
+        <link_name>battery_link</link_name>
+        <battery_name>battery</battery_name>
         <open_circuit_voltage_constant_coef>${open_circuit_voltage_constant_coef}</open_circuit_voltage_constant_coef>
         <open_circuit_voltage_linear_coef>${open_circuit_voltage_linear_coef}</open_circuit_voltage_linear_coef>

File: uuv-simulator/uuv_gazebo_plugins/uuv_gazebo_ros_plugins/urdf/fin_snippets.xacro (robot description, xacro)
@@ -20,12 +20,12 @@
             cda_stall
             current_velocity_topic">
-    <joint name="${namespace}/fin${fin_id}_joint" type="revolute">
+    <joint name="fin${fin_id}_joint" type="revolute">
         <limit effort="0" lower="${min_joint_limit}" upper="${max_joint_limit}" velocity="0"/>
         <xacro:insert_block name="origin"/>
         <axis xyz="0 0 1"/>
         <parent link="${parent_link}" />
-        <child link="${namespace}/fin${fin_id}" />
+        <child link="fin${fin_id}" />
     </joint>
-    <link name="${namespace}/fin${fin_id}">
+    <link name="fin${fin_id}">
       <xacro:no_inertial />
       <visual>
@@ -55,6 +55,6 @@
         <current_velocity_topic>${current_velocity_topic}</current_velocity_topic>
         <fin_id>${fin_id}</fin_id>
-        <link_name>${namespace}/fin${fin_id}</link_name>
-        <joint_name>${namespace}/fin${fin_id}_joint</joint_name>
+        <link_name>fin${fin_id}</link_name>
+        <joint_name>fin${fin_id}_joint</joint_name>
       </plugin>
     </gazebo>
@@ -73,12 +73,12 @@
             drag_constant
             current_velocity_topic">
-    <joint name="${namespace}/fin${fin_id}_joint" type="revolute">
+    <joint name="fin${fin_id}_joint" type="revolute">
         <limit effort="0" lower="${min_joint_limit}" upper="${max_joint_limit}" velocity="0"/>
         <xacro:insert_block name="origin"/>
         <axis xyz="0 0 1"/>
         <parent link="${parent_link}" />
-        <child link="${namespace}/fin${fin_id}" />
+        <child link="fin${fin_id}" />
     </joint>
-    <link name="${namespace}/fin${fin_id}">
+    <link name="fin${fin_id}">
       <xacro:no_inertial />
       <visual>
@@ -102,6 +102,6 @@
         <current_velocity_topic>${current_velocity_topic}</current_velocity_topic>
         <fin_id>${fin_id}</fin_id>
-        <link_name>${namespace}/fin${fin_id}</link_name>
-        <joint_name>${namespace}/fin${fin_id}_joint</joint_name>
+        <link_name>fin${fin_id}</link_name>
+        <joint_name>fin${fin_id}_joint</joint_name>
       </plugin>
     </gazebo>

File: uuv-simulator/uuv_gazebo_plugins/uuv_gazebo_ros_plugins/urdf/thruster_snippets.xacro (robot description, xacro)
@@ -76,11 +76,11 @@
             *dynamics
             *conversion">
-    <joint name="${namespace}/thruster_${thruster_id}_joint" type="continuous">
+    <joint name="thruster_${thruster_id}_joint" type="continuous">
       <xacro:insert_block name="origin"/>
       <axis xyz="1 0 0"/>
-      <parent link="${namespace}/base_link"/>
-      <child link="${namespace}/thruster_${thruster_id}"/>
+      <parent link="base_link"/>
+      <child link="thruster_${thruster_id}"/>
     </joint>
-    <link name="${namespace}/thruster_${thruster_id}">
+    <link name="thruster_${thruster_id}">
       <xacro:box_inertial x="0.1" y="0.1" z="0.1" mass="0.3">
         <origin xyz="0 0 0" rpy="0 0 0"/>
@@ -103,6 +103,6 @@
     <gazebo>
       <plugin name="${namespace}_${thruster_id}_thruster_model" filename="libthruster_ros_plugin.so">
-        <linkName>${namespace}/thruster_${thruster_id}</linkName>
-        <jointName>${namespace}/thruster_${thruster_id}_joint</jointName>
+        <linkName>thruster_${thruster_id}</linkName>
+        <jointName>thruster_${thruster_id}_joint</jointName>
         <thrusterID>${thruster_id}</thrusterID>
         <xacro:insert_block name="dynamics"/>
@@ -111,5 +111,5 @@
     </gazebo>
    <!-- Choose thruster color -->
-    <gazebo reference="${namespace}/thruster_${thruster_id}">
+    <gazebo reference="thruster_${thruster_id}">
       <selfCollide>false</selfCollide>
     <material>Gazebo/Red</material>

File: uuv-simulator/uuv_sensor_plugins/uuv_sensor_ros_plugins/urdf/camera_snippets.xacro (robot description, xacro)
@@ -61,5 +61,5 @@
       *inertia *origin">
     <!-- Sensor link -->
-    <link name="${namespace}/camera${suffix}_link">
+    <link name="camera${suffix}_link">
       <inertial>
         <xacro:insert_block name="inertia" />
@@ -74,12 +74,12 @@
       <xacro:no_collision/>
     </link>
-    <joint name="${namespace}/camera${suffix}_joint" type="revolute">
+    <joint name="camera${suffix}_joint" type="revolute">
       <xacro:insert_block name="origin" />
       <parent link="${parent_link}" />
-      <child link="${namespace}/camera${suffix}_link" />
+      <child link="camera${suffix}_link" />
       <limit upper="0" lower="0" effort="0" velocity="0" />
       <axis xyz="1 0 0"/>
     </joint>
-    <link name="${namespace}/camera${suffix}_link_optical">
+    <link name="camera${suffix}_link_optical">
       <xacro:box_inertial x="0.0001" y="0.0001" z="0.0001" mass="0.001">
         <origin xyz="0 0 0" rpy="0 0 0"/>
@@ -99,12 +99,12 @@
       </visual>
     </link>
-    <joint name="${namespace}/camera${suffix}_optical_joint" type="revolute">
+    <joint name="camera${suffix}_optical_joint" type="revolute">
       <origin xyz="0 0 0" rpy="${-pi/2} 0 ${-pi/2}"/>
-      <parent link="${namespace}/camera${suffix}_link"/>
-      <child link="${namespace}/camera${suffix}_link_optical"/>
+      <parent link="camera${suffix}_link"/>
+      <child link="camera${suffix}_link_optical"/>
       <limit upper="0" lower="0" effort="0" velocity="0" />
       <axis xyz="1 0 0"/>
     </joint>
-    <gazebo reference="${namespace}/camera${suffix}_link">
+    <gazebo reference="camera${suffix}_link">
       <sensor type="camera" name="camera${suffix}">
         <update_rate>${update_rate}</update_rate>
@@ -151,5 +151,5 @@
       *inertia *origin">
     <!-- Sensor link -->
-    <link name="${namespace}/camera${suffix}_link">
+    <link name="camera${suffix}_link">
       <inertial>
         <xacro:insert_block name="inertia" />
@@ -164,12 +164,12 @@
       <xacro:no_collision/>
     </link>
-    <joint name="${namespace}/camera${suffix}_joint" type="revolute">
+    <joint name="camera${suffix}_joint" type="revolute">
       <xacro:insert_block name="origin" />
       <parent link="${parent_link}" />
-      <child link="${namespace}/camera${suffix}_link" />
+      <child link="camera${suffix}_link" />
       <axis xyz="1 0 0"/>
       <limit upper="0" lower="0" effort="0" velocity="0" />
     </joint>
-    <gazebo reference="${namespace}/camera${suffix}_link">
+    <gazebo reference="camera${suffix}_link">
       <sensor type="depth" name="camera${suffix}">
         <update_rate>${update_rate}</update_rate>
@@ -194,5 +194,5 @@
           <updateRate>${update_rate}</updateRate>
           <cameraName>$camera${suffix}</cameraName>
-          <frameName>${namespace}/camera${suffix}_link</frameName>
+          <frameName>camera${suffix}_link</frameName>
           <attenuationR>0.01</attenuationR>
           <attenuationG>0.01</attenuationG>

File: uuv-simulator/uuv_sensor_plugins/uuv_sensor_ros_plugins/urdf/chemical_concentration_snippets.xacro (robot description, xacro)
@@ -81,5 +81,5 @@
             salinity_output_topic salinity_unit gain noise_sigma noise_amplitude">
     <!-- Sensor link -->
-   <link name="${namespace}/cc_sensor_link">
+   <link name="cc_sensor_link">
      <inertial>
        <inertia ixx="0.00001" ixy="0.0" ixz="0.0" iyy="0.00001" iyz="0.0" izz="0.00001" />
@@ -88,8 +88,8 @@
      </inertial>
    </link>
-   <joint name="${namespace}/cc_sensor_joint" type="revolute">
+   <joint name="cc_sensor_joint" type="revolute">
      <xacro:insert_block name="origin" />
      <parent link="${parent_link}" />
-     <child link="${namespace}/cc_sensor_link" />
+     <child link="cc_sensor_link" />
      <axis xyz="1 0 0"/>
      <limit upper="0" lower="0" effort="0" velocity="0" />
@@ -99,5 +99,5 @@
        name="particle_concentration{suffix}_sensor">
        <robot_namespace>${namespace}</robot_namespace>
-       <link_name>${namespace}/cc_sensor_link</link_name>
+       <link_name>cc_sensor_link</link_name>
        <plume_topic>${input_topic}</plume_topic>
        <sensor_topic>${output_topic}</sensor_topic>

File: uuv-simulator/uuv_sensor_plugins/uuv_sensor_ros_plugins/urdf/dvl_snippets.xacro (robot description, xacro)
@@ -69,5 +69,5 @@
   </xacro:macro>
   <xacro:macro name="dvl_single_sonar" params="namespace suffix index pitch yaw">
-    <link name="${namespace}/dvl${suffix}_sonar${index}_link">
+    <link name="dvl${suffix}_sonar${index}_link">
       <inertial>
         <mass value="0.001" />  <!-- [kg] -->
@@ -77,12 +77,12 @@
       <xacro:no_collision/>
     </link>
-    <joint name="${namespace}/dvl${suffix}_sonar${index}_joint" type="revolute">
+    <joint name="dvl${suffix}_sonar${index}_joint" type="revolute">
       <origin xyz="0 0 0" rpy="0 ${pitch} ${yaw}"/>
-      <parent link="${namespace}/dvl${suffix}_link" />
-      <child link="${namespace}/dvl${suffix}_sonar${index}_link" />
+      <parent link="dvl${suffix}_link" />
+      <child link="dvl${suffix}_sonar${index}_link" />
       <limit upper="0" lower="0" effort="0" velocity="0" />
       <axis xyz="1 0 0"/>
     </joint>
-    <gazebo reference="${namespace}/dvl${suffix}_sonar${index}_link">
+    <gazebo reference="dvl${suffix}_sonar${index}_link">
       <sensor type="ray" name="dvl${suffix}_sonar${index}">
         <pose>0 0 0 0 0 0</pose>
@@ -115,5 +115,5 @@
           <updateRate>1</updateRate>
           <topicName>${topic}_sonar${index}</topicName>
-          <frameName>${namespace}/dvl${suffix}_sonar${index}_link</frameName>
+          <frameName>dvl${suffix}_sonar${index}_link</frameName>
           <fov>0.06</fov>
           <radiation>ultrasound</radiation>
@@ -125,5 +125,5 @@
     params="namespace suffix parent_link topic scale *origin update_rate
     reference_frame noise_sigma noise_amplitude">
-    <link name="${namespace}/dvl${suffix}_link">
+    <link name="dvl${suffix}_link">
       <inertial>
         <mass value="0.001" />  <!-- [kg] -->
@@ -138,8 +138,8 @@
       <xacro:no_collision/>
     </link>
-    <joint name="${namespace}/dvl${suffix}_joint" type="revolute">
+    <joint name="dvl${suffix}_joint" type="revolute">
       <xacro:insert_block name="origin" />
       <parent link="${parent_link}" />
-      <child link="${namespace}/dvl${suffix}_link" />
+      <child link="dvl${suffix}_link" />
       <limit upper="0" lower="0" effort="0" velocity="0" />
       <axis xyz="1 0 0"/>
@@ -165,5 +165,5 @@
         <robot_namespace>${namespace}</robot_namespace> <!-- (string, required): ros namespace in which the messages are published -->
 	<!-- Changed from dvl_link to base_link to get ENU coordinate frame -->
-        <link_name>${namespace}/base_link</link_name> <!-- (string, required): name of the body which holds the IMU sensor -->
+        <link_name>base_link</link_name> <!-- (string, required): name of the body which holds the IMU sensor -->
         <sensor_topic>${topic}</sensor_topic> <!-- (string): name of the sensor output topic and prefix of service names -->
         <update_rate>${update_rate}</update_rate> <!-- Update period [s] -->
@@ -174,8 +174,8 @@
         <static_reference_frame>${reference_frame}</static_reference_frame>
         <!-- Declaring the beams -->
-        <beam_link_name_0>${namespace}/dvl_sonar0_link</beam_link_name_0>
-        <beam_link_name_1>${namespace}/dvl_sonar1_link</beam_link_name_1>
-        <beam_link_name_2>${namespace}/dvl_sonar2_link</beam_link_name_2>
-        <beam_link_name_3>${namespace}/dvl_sonar3_link</beam_link_name_3>
+        <beam_link_name_0>dvl_sonar0_link</beam_link_name_0>
+        <beam_link_name_1>dvl_sonar1_link</beam_link_name_1>
+        <beam_link_name_2>dvl_sonar2_link</beam_link_name_2>
+        <beam_link_name_3>dvl_sonar3_link</beam_link_name_3>
         <!-- Declaring the beam output topics -->
         <beam_topic_0>${topic}_sonar0</beam_topic_0>

File: uuv-simulator/uuv_sensor_plugins/uuv_sensor_ros_plugins/urdf/gps_sensor_snippets.xacro (robot description, xacro)
@@ -18,5 +18,5 @@
     vertical_vel_std_dev *inertia *origin update_rate">
       <!-- GPS link -->
-     <link name="${namespace}/gps_link">
+     <link name="gps_link">
        <inertial>
          <inertia ixx="0.00001" ixy="0.0" ixz="0.0" iyy="0.00001" iyz="0.0" izz="0.00001" />
@@ -31,13 +31,13 @@
      </link>
      <!-- GPS joint -->
-    <joint name="${namespace}/gps_joint" type="revolute">
+    <joint name="gps_joint" type="revolute">
       <xacro:insert_block name="origin" />
       <parent link="${parent_link}" />
-      <child link="${namespace}/gps_link" />
+      <child link="gps_link" />
       <axis xyz="1 0 0"/>
       <limit upper="0" lower="0" effort="0" velocity="0" />
     </joint>
-    <gazebo reference="${namespace}/gps_link">
-      <sensor type="gps" name="${namespace}/gps">
+    <gazebo reference="gps_link">
+      <sensor type="gps" name="gps">
         <pose>0 0 0 0 0 0</pose>
         <visualize>0</visualize>

File: uuv-simulator/uuv_sensor_plugins/uuv_sensor_ros_plugins/urdf/imu_snippets.xacro (robot description, xacro)
@@ -123,5 +123,5 @@
       *inertia *origin">
     <!-- IMU link -->
-    <link name="${namespace}/imu${imu_suffix}_link">
+    <link name="imu${imu_suffix}_link">
       <xacro:box_inertial x="0.0001" y="0.0001" z="0.0001" mass="${mass_imu_sensor}">
         <origin xyz="0 0 0" rpy="0 0 0"/>
@@ -135,8 +135,8 @@
     </link>
     <!-- IMU joint -->
-    <joint name="${namespace}/imu${imu_suffix}_joint" type="revolute">
+    <joint name="imu${imu_suffix}_joint" type="revolute">
       <xacro:insert_block name="origin" />
       <parent link="${parent_link}" />
-      <child link="${namespace}/imu${imu_suffix}_link" />
+      <child link="imu${imu_suffix}_link" />
       <limit upper="0" lower="0" effort="0" velocity="0" />
       <axis xyz="1 0 0"/>
@@ -147,5 +147,5 @@
            https://github.com/ethz-asl/kalibr/wiki/IMU-Noise-Model-and-Intrinsics -->
         <robot_namespace>${namespace}</robot_namespace> <!-- (string, required): ros namespace in which the messages are published -->
-        <link_name>${namespace}/imu${imu_suffix}_link</link_name> <!-- (string, required): name of the body which holds the IMU sensor -->
+        <link_name>imu${imu_suffix}_link</link_name> <!-- (string, required): name of the body which holds the IMU sensor -->
         <sensor_topic>${imu_topic}</sensor_topic> <!-- (string): name of the sensor output topic and prefix of service names (defaults to imu) -->
         <gyroscope_noise_density>${gyroscope_noise_density}</gyroscope_noise_density> <!-- Gyroscope noise density (two-sided spectrum) [rad/s/sqrt(Hz)] -->
