Commit message: remove all known instances of tf prefixing

File: uuv-simulator/uuv_sensor_plugins/uuv_sensor_ros_plugins/urdf/magnetometer_snippets.xacro (robot description, xacro)
@@ -46,5 +46,5 @@
       *inertia *origin">
     <!-- Sensor link -->
-    <link name="${namespace}/magnetometer${suffix}_link">
+    <link name="magnetometer${suffix}_link">
       <inertial>
         <xacro:insert_block name="inertia" />
@@ -60,8 +60,8 @@
     </link>
     <!-- Sensor joint -->
-    <joint name="${namespace}/magnetometer${suffix}_joint" type="revolute">
+    <joint name="magnetometer${suffix}_joint" type="revolute">
       <xacro:insert_block name="origin" />
       <parent link="${parent_link}" />
-      <child link="${namespace}/magnetometer${suffix}_link" />
+      <child link="magnetometer${suffix}_link" />
       <limit upper="0" lower="0" effort="0" velocity="0" />
       <axis xyz="1 0 0"/>
@@ -70,5 +70,5 @@
       <plugin filename="libuuv_gazebo_ros_magnetometer_plugin.so" name="libuuv_gazebo_ros_magnetometer_${suffix}_plugin">
         <robot_namespace>${namespace}</robot_namespace> <!-- (string, required): ros namespace in which the messages are published -->
-        <link_name>${namespace}/magnetometer${suffix}_link</link_name> <!-- (string, required): name of the body which holds the IMU sensor -->
+        <link_name>magnetometer${suffix}_link</link_name> <!-- (string, required): name of the body which holds the IMU sensor -->
         <sensor_topic>${topic}</sensor_topic> <!-- (string): name of the sensor output topic and prefix of service names (defaults to imu) -->
         <update_rate>${update_rate}</update_rate> <!-- Update period of accelerometer and gyroscope [s] -->

File: uuv-simulator/uuv_sensor_plugins/uuv_sensor_ros_plugins/urdf/pose_3d_snippets.xacro (robot description, xacro)
@@ -16,5 +16,5 @@
     update_rate *origin noise_sigma reference_frame publish_ned_odom noise_amplitude">
     <!-- Mount a 3D pose sensor -->
-    <link name="${namespace}/pose_sensor_link_${suffix}">
+    <link name="pose_sensor_link_${suffix}">
       <inertial>
         <inertia ixx="0.00001" ixy="0.0" ixz="0.0" iyy="0.00001" iyz="0.0" izz="0.00001" />
@@ -28,9 +28,9 @@
       </visual>
     </link>
-    <joint name="${namespace}/pose_sensor_${suffix}_joint" type="revolute">
+    <joint name="pose_sensor_${suffix}_joint" type="revolute">
       <xacro:insert_block name="origin" />
       <axis xyz="0 0 1"/>
       <parent link="${parent_link}"/>
-      <child link="${namespace}/pose_sensor_link_${suffix}"/>
+      <child link="pose_sensor_link_${suffix}"/>
       <limit effort="0" lower="0" upper="0" velocity="0"/>
     </joint>
@@ -38,5 +38,5 @@
       <plugin name="pose_3d_plugin" filename="libuuv_gazebo_ros_pose_gt_plugin.so">
         <robot_namespace>${namespace}</robot_namespace>
-        <link_name>${namespace}/base_link</link_name>
+        <link_name>base_link</link_name>
         <sensor_topic>${topic}</sensor_topic>
         <static_reference_frame>${reference_frame}</static_reference_frame>

File: uuv-simulator/uuv_sensor_plugins/uuv_sensor_ros_plugins/urdf/pressure_snippets.xacro (robot description, xacro)
@@ -63,5 +63,5 @@
       range noise_sigma noise_amplitude estimateDepth depthTopic standardPressure kPaPerM
       *inertia *origin">
-    <link name="${namespace}/pressure${suffix}_link">
+    <link name="pressure${suffix}_link">
       <inertial>
         <xacro:insert_block name="inertia" />
@@ -76,8 +76,8 @@
       <xacro:no_collision/>
     </link>
-    <joint name="${namespace}/pressure${suffix}_joint" type="revolute">
+    <joint name="pressure${suffix}_joint" type="revolute">
       <xacro:insert_block name="origin" />
       <parent link="${parent_link}" />
-      <child link="${namespace}/pressure${suffix}_link" />
+      <child link="pressure${suffix}_link" />
       <limit upper="0" lower="0" effort="0" velocity="0" />
       <axis xyz="1 0 0"/>
@@ -86,5 +86,5 @@
       <plugin filename="libuuv_gazebo_ros_subsea_pressure_plugin.so" name="libuuv_gazebo_subseapressure${suffix}_plugin">
         <robot_namespace>${namespace}</robot_namespace> <!-- (string, required): ros namespace in which the messages are published -->
-        <link_name>${namespace}/pressure${suffix}_link</link_name> <!-- (string, required): name of the body which holds the IMU sensor -->
+        <link_name>pressure${suffix}_link</link_name> <!-- (string, required): name of the body which holds the IMU sensor -->
         <sensor_topic>${topic}</sensor_topic> <!-- (string): name of the sensor output topic and prefix of service names (defaults to imu) -->
         <update_rate>${update_rate}</update_rate> <!-- Update period of accelerometer and gyroscope [s] -->

File: uuv-simulator/uuv_sensor_plugins/uuv_sensor_ros_plugins/urdf/rpt_snippets.xacro (robot description, xacro)
@@ -35,5 +35,5 @@
     params="namespace suffix parent_link topic noise_sigma noise_amplitude
     *origin">
-    <link name="${namespace}/rpt${suffix}_link">
+    <link name="rpt${suffix}_link">
       <inertial>
         <mass value="0.001" />  <!-- [kg] -->
@@ -48,8 +48,8 @@
       <xacro:no_collision/>
     </link>
-    <joint name="${namespace}/rpt${suffix}_joint" type="revolute">
+    <joint name="rpt${suffix}_joint" type="revolute">
       <xacro:insert_block name="origin" />
       <parent link="${parent_link}" />
-      <child link="${namespace}/rpt${suffix}_link" />
+      <child link="rpt${suffix}_link" />
       <limit upper="0" lower="0" effort="0" velocity="0" />
       <axis xyz="1 0 0"/>
@@ -58,5 +58,5 @@
       <plugin filename="libuuv_gazebo_ros_rpt_plugin.so" name="libuuv_gazebo_rpt${suffix}_plugin">
         <robot_namespace>${namespace}</robot_namespace> <!-- ros namespace in which the messages are published -->
-        <link_name>${namespace}/rpt${suffix}_link</link_name> <!-- sensor link name -->
+        <link_name>rpt${suffix}_link</link_name> <!-- sensor link name -->
         <static_reference_frame>ssbl</static_reference_frame> <!-- name of the refernce frame of all position measurements -->
         <sensor_topic>${topic}</sensor_topic> <!-- name of the sensor output topic and prefix of service name -->

File: uuv-simulator/uuv_sensor_plugins/uuv_sensor_ros_plugins/urdf/sonar_snippets.xacro (robot description, xacro)
@@ -99,5 +99,5 @@
       *inertia *origin *visual">
     <!-- Sensor link -->
-    <link name="${namespace}/sonar${suffix}_link">
+    <link name="sonar${suffix}_link">
       <inertial>
         <xacro:insert_block name="inertia" />
@@ -111,9 +111,9 @@
     <xacro:insert_block name="origin" />
     <parent link="${parent_link}" />
-    <child link="${namespace}/sonar${suffix}_link" />
+    <child link="sonar${suffix}_link" />
     <limit upper="0" lower="0" effort="0" velocity="0" />
     <axis xyz="1 0 0"/>
   </joint>
-  <gazebo reference="${namespace}/sonar${suffix}_link">
+  <gazebo reference="sonar${suffix}_link">
     <sensor type="gpu_ray" name="sonar${suffix}">
       <pose>0 0 0 0 0 0</pose>

File: uuv-simulator/uuv_sensor_plugins/uuv_sensor_ros_plugins/urdf/stereo_snippets.xacro (robot description, xacro)
@@ -34,5 +34,5 @@
   </xacro:macro>
   <xacro:macro name="duo3d_camera" params="namespace parent_link *origin">
-    <link name="${namespace}/duo3d_left_link">
+    <link name="duo3d_left_link">
       <inertial>
         <mass value="0.01"/>
@@ -46,12 +46,12 @@
       <xacro:no_collision/>
     </link>
-    <joint name="${namespace}/duo3d_joint" type="revolute">
+    <joint name="duo3d_joint" type="revolute">
       <xacro:insert_block name="origin" />
       <parent link="${parent_link}" />
-      <child link="${namespace}/duo3d_left_link" />
+      <child link="duo3d_left_link" />
       <limit upper="0" lower="0" effort="0" velocity="0" />
       <axis xyz="1 0 0"/>
     </joint>
-    <gazebo reference="${namespace}/duo3d_left_link">
+    <gazebo reference="duo3d_left_link">
       <sensor name="camera" type="camera">
       <camera>
@@ -78,8 +78,8 @@
         <alwaysOn>true</alwaysOn>
         <updateRate>30.0</updateRate>
-        <cameraName>${namespace}/duo3d_left</cameraName>
+        <cameraName>duo3d_left</cameraName>
         <imageTopicName>image_raw</imageTopicName>
         <cameraInfoTopicName>camera_info</cameraInfoTopicName>
-        <frameName>${namespace}/duo3d_left_link</frameName>
+        <frameName>duo3d_left_link</frameName>
         <hackBaseline>0.07</hackBaseline>
         <distortionK1>${k1l}</distortionK1>
@@ -94,5 +94,5 @@
     </sensor>
     </gazebo>
-    <link name="${namespace}/duo3d_right_link">
+    <link name="duo3d_right_link">
       <inertial>
         <mass value="0.01"/>
@@ -101,12 +101,12 @@
       <xacro:no_collision/>
     </link>
-    <joint name="${namespace}/duo3d_right_joint" type="revolute">
+    <joint name="duo3d_right_joint" type="revolute">
       <origin xyz="0.0 -0.03 0" rpy="0 0 0"/>
-      <parent link="${namespace}/duo3d_left_link" />
-      <child link="${namespace}/duo3d_right_link" />
+      <parent link="duo3d_left_link" />
+      <child link="duo3d_right_link" />
       <limit upper="0" lower="0" effort="0" velocity="0" />
       <axis xyz="1 0 0"/>
     </joint>
-    <gazebo reference="${namespace}/duo3d_right_link">
+    <gazebo reference="duo3d_right_link">
       <sensor name="camera" type="camera">
       <camera>
@@ -133,8 +133,8 @@
         <alwaysOn>true</alwaysOn>
         <updateRate>30.0</updateRate>
-        <cameraName>${namespace}/duo3d_right</cameraName>
+        <cameraName>duo3d_right</cameraName>
         <imageTopicName>image_raw</imageTopicName>
         <cameraInfoTopicName>camera_info</cameraInfoTopicName>
-        <frameName>${namespace}/duo3d_right_link</frameName>
+        <frameName>duo3d_right_link</frameName>
         <hackBaseline>0.07</hackBaseline>
         <distortionK1>${k1l}</distortionK1>

Commit message: controller cleanup

File: tauv_config/albatross_description/urdf/base.xacro (robot description, xacro)
@@ -27,5 +27,5 @@
   this geometry as simple as possible to improve the performance the physics engine
   regarding the computation of collision forces) -->
-  <xacro:property name="collision_mesh_file" value="file://$(find albatross_description)/meshes/vehicle.stl"/>
+  <xacro:property name="collision_mesh_file" value="file://$(find albatross_description)/meshes/vehicle.dae"/>
   <!-- Vehicle macro -->
   <xacro:macro name="albatross_base" params="namespace *gazebo">

File: tauv_config/albatross_description/urdf/gazebo.xacro (robot description, xacro)
@@ -4,5 +4,5 @@
     <xacro:property name="albatross_cob" value="0 0 0"/>
     <!-- Vehicle's actual volume (Gazebo cannot compute the volume out of the mesh) -->
-    <xacro:property name="albatross_volume" value="0.01854"/>
+    <xacro:property name="albatross_volume" value="0.016"/>
     <!-- Describing the dimensions of the vehicle's bounding box -->
     <xacro:property name="albatross_length" value="1"/>
