Commit message: thrusters spinning from wrench inputs. TAM or inversion matrix is wrong

File: tauv_config/albatross_description/urdf/sensors.xacro (robot description, xacro)
@@ -29,5 +29,5 @@
   <!-- IMU  -->
   <xacro:default_imu namespace="${namespace}" parent_link="${namespace}/base_link">
-    <origin xyz="0 0 0" rpy="0 0 0"/>
+    <origin xyz="0 0 0" rpy="${0} ${90*d2r} ${-90*d2r}"/>
   </xacro:default_imu>
   <!-- Mount a camera  -->

Commit message: added stereo into sim, changed to sandy bottom

File: tauv_config/albatross_description/urdf/sensors.xacro (robot description, xacro)
@@ -35,6 +35,9 @@
     <origin xyz="0.29 0.0 0." rpy="0 0 0"/>
   </xacro:default_camera>
-  <xacro:default_camera namespace="${namespace}" parent_link="${namespace}/base_link" suffix="under">
-    <origin xyz="0.15 0.0 -0.06" rpy="0 ${0.5*pi} 0"/>
+  <xacro:default_camera namespace="${namespace}" parent_link="${namespace}/base_link" suffix="under1">
+    <origin xyz="0.15 0.05 -0.06" rpy="0 ${0.5*pi} 0"/>
   </xacro:default_camera>
+  <xacro:default_camera namespace="${namespace}" parent_link="${namespace}/base_link" suffix="under2">
+      <origin xyz="0.15 -0.05 -0.06" rpy="0 ${0.5*pi} 0"/>
+    </xacro:default_camera>
 </robot>

Commit message: publishes shady tf and odom

File: tauv_config/albatross_description/urdf/sensors.xacro (robot description, xacro)
@@ -27,7 +27,10 @@
     <origin xyz="0 0 0" rpy="0 0 0"/>
   </xacro:default_pressure>
+  <xacro:default_camera namespace="${namespace}" parent_link="base_link" suffix="under2">
+    <origin xyz="0.15 -0.05 -0.06" rpy="0 ${0.5*pi} 0"/>
+  </xacro:default_camera>
   <!-- IMU  -->
   <xacro:default_imu namespace="${namespace}" parent_link="base_link">
-    <origin xyz="0 0 0" rpy="${0} ${90*d2r} ${-90*d2r}"/>
+    <origin xyz="0 0 0" rpy="${0} ${0} ${0}"/>
   </xacro:default_imu>
   <!-- Mount a camera -->
@@ -38,6 +41,3 @@
     <origin xyz="0.15 0.05 -0.06" rpy="0 ${0.5*pi} 0"/>
   </xacro:default_camera>
-  <xacro:default_camera namespace="${namespace}" parent_link="base_link" suffix="under2">
-      <origin xyz="0.15 -0.05 -0.06" rpy="0 ${0.5*pi} 0"/>
-    </xacro:default_camera>
 </robot>

Commit message: fix xacro

File: tauv_config/albatross_description/urdf/sensors.xacro (robot description, xacro)
@@ -32,5 +32,5 @@
   <!-- IMU  -->
   <xacro:default_imu namespace="${namespace}" parent_link="base_link">
-    <origin xyz="0 0 0" rpy="${0} ${0} ${0}"/>
+    <origin xyz="0 0 0" rpy="${0} ${0.5*pi} ${0.5*pi}"/>
   </xacro:default_imu>
   <!-- Mount a camera -->

Commit message: fix xacro more

File: tauv_config/albatross_description/urdf/sensors.xacro (robot description, xacro)
@@ -32,5 +32,5 @@
   <!-- IMU  -->
   <xacro:default_imu namespace="${namespace}" parent_link="base_link">
-    <origin xyz="0 0 0" rpy="${0} ${0.5*pi} ${0.5*pi}"/>
+    <origin xyz="0 0 0" rpy="${0} ${0.5*pi} ${-0.5*pi}"/>
   </xacro:default_imu>
   <!-- Mount a camera -->

Commit message: imu urdf level

File: tauv_config/albatross_description/urdf/sensors.xacro (robot description, xacro)
@@ -32,5 +32,5 @@
   <!-- IMU  -->
   <xacro:default_imu namespace="${namespace}" parent_link="base_link">
-    <origin xyz="0 0 0" rpy="${0} ${0.5*pi} ${-0.5*pi}"/>
+    <origin xyz="0 0 0" rpy="${0} ${0} ${0}"/>
   </xacro:default_imu>
   <!-- Mount a camera -->

Commit message: changed imu urdf

File: tauv_config/albatross_description/urdf/sensors.xacro (robot description, xacro)
@@ -32,5 +32,5 @@
   <!-- IMU  -->
   <xacro:default_imu namespace="${namespace}" parent_link="base_link">
-    <origin xyz="0 0 0" rpy="${0} ${0} ${0}"/>
+    <origin xyz="0 0 0" rpy="${0} ${.5*pi} ${.5*pi}"/>
   </xacro:default_imu>
   <!-- Mount a camera -->

Commit message: reverted imu pos

File: tauv_config/albatross_description/urdf/sensors.xacro (robot description, xacro)
@@ -32,5 +32,5 @@
   <!-- IMU  -->
   <xacro:default_imu namespace="${namespace}" parent_link="base_link">
-    <origin xyz="0 0 0" rpy="${0} ${.5*pi} ${.5*pi}"/>
+    <origin xyz="0 0 0" rpy="${0} ${0} ${0}"/>
   </xacro:default_imu>
   <!-- Mount a camera -->

Commit message: urdf

File: tauv_config/albatross_description/urdf/sensors.xacro (robot description, xacro)
@@ -32,5 +32,5 @@
   <!-- IMU  -->
   <xacro:default_imu namespace="${namespace}" parent_link="base_link">
-    <origin xyz="0 0 0" rpy="${0} ${.5*pi} ${.5*pi}"/>
+    <origin xyz="0 0 0" rpy="${0} ${.5*pi} ${-.5*pi}"/>
   </xacro:default_imu>
   <!-- Mount a camera -->

Commit message: urdf back

File: tauv_config/albatross_description/urdf/sensors.xacro (robot description, xacro)
@@ -32,5 +32,5 @@
   <!-- IMU  -->
   <xacro:default_imu namespace="${namespace}" parent_link="base_link">
-    <origin xyz="0 0 0" rpy="${0} ${.5*pi} ${-.5*pi}"/>
+    <origin xyz="0 0 0" rpy="${0} ${0} ${0}"/>
   </xacro:default_imu>
   <!-- Mount a camera -->

Commit message: added yaw to imu

File: tauv_config/albatross_description/urdf/sensors.xacro (robot description, xacro)
@@ -32,5 +32,5 @@
   <!-- IMU  -->
   <xacro:default_imu namespace="${namespace}" parent_link="base_link">
-    <origin xyz="0 0 0" rpy="${0} ${0} ${0}"/>
+    <origin xyz="0 0 0" rpy="${0} ${0} ${.5*pi}"/>
   </xacro:default_imu>
   <!-- Mount a camera -->

Commit message: IMU regular now

File: tauv_config/albatross_description/urdf/sensors.xacro (robot description, xacro)
@@ -32,5 +32,5 @@
   <!-- IMU  -->
   <xacro:default_imu namespace="${namespace}" parent_link="base_link">
-    <origin xyz="0 0 0" rpy="${0} ${0} ${.5*pi}"/>
+    <origin xyz="0 0 0" rpy="${0} ${0} ${0}"/>
   </xacro:default_imu>
   <!-- Mount a camera -->

Commit message: pls

File: tauv_config/albatross_description/urdf/sensors.xacro (robot description, xacro)
@@ -32,5 +32,5 @@
   <!-- IMU  -->
   <xacro:default_imu namespace="${namespace}" parent_link="base_link">
-    <origin xyz="0 0 0" rpy="${0} ${0} ${.5*pi}"/>
+    <origin xyz="0 0 0" rpy="${0} ${.5*pi} ${.5*pi}"/>
   </xacro:default_imu>
   <!-- Mount a camera -->

Commit message: no p

File: tauv_config/albatross_description/urdf/sensors.xacro (robot description, xacro)
@@ -32,5 +32,5 @@
   <!-- IMU  -->
   <xacro:default_imu namespace="${namespace}" parent_link="base_link">
-    <origin xyz="0 0 0" rpy="${0} ${.5*pi} ${.5*pi}"/>
+    <origin xyz="0 0 0" rpy="${0} ${0} ${.5*pi}"/>
   </xacro:default_imu>
   <!-- Mount a camera -->

Commit message: running stereo_image_proc on downward cameras

File: tauv_config/albatross_description/urdf/sensors.xacro (robot description, xacro)
@@ -27,5 +27,5 @@
     <origin xyz="0 0 0" rpy="0 0 0"/>
   </xacro:default_pressure>
-  <xacro:default_camera namespace="${namespace}" parent_link="base_link" suffix="under2">
+  <xacro:default_camera namespace="${namespace}" parent_link="base_link" suffix="_under_stereo_left">
     <origin xyz="0.15 -0.05 -0.06" rpy="0 ${0.5*pi} 0"/>
   </xacro:default_camera>
@@ -35,9 +35,12 @@
   </xacro:default_imu>
   <!-- Mount a camera -->
-  <xacro:default_camera namespace="${namespace}" parent_link="base_link" suffix="front">
-    <origin xyz="0.29 0.0 0." rpy="0 0 0"/>
+  <xacro:default_camera namespace="${namespace}" parent_link="base_link" suffix="_front_stereo_left">
+    <origin xyz="0.29 -0.10 0." rpy="0 0 0"/>
   </xacro:default_camera>
-  <xacro:default_camera namespace="${namespace}" parent_link="base_link" suffix="under1">
-    <origin xyz="0.15 0.05 -0.06" rpy="0 ${0.5*pi} 0"/>
+  <xacro:default_camera namespace="${namespace}" parent_link="base_link" suffix="_front_stereo_right">
+    <origin xyz="0.29 .05 0." rpy="0 0 0"/>
+  </xacro:default_camera>
+  <xacro:default_camera namespace="${namespace}" parent_link="base_link" suffix="_under_stereo_right">
+    <origin xyz="0.15 0.10 -0.06" rpy="0 ${0.5*pi} 0"/>
   </xacro:default_camera>
 </robot>

Commit message: removed imu_complementary filter dependency, we are using madgwick filter

File: tauv_config/albatross_description/urdf/sensors.xacro (robot description, xacro)
@@ -27,7 +27,4 @@
     <origin xyz="0 0 0" rpy="0 0 0"/>
   </xacro:default_pressure>
-  <xacro:default_camera namespace="${namespace}" parent_link="base_link" suffix="_under_stereo_left">
-    <origin xyz="0.15 -0.05 -0.06" rpy="0 ${0.5*pi} 0"/>
-  </xacro:default_camera>
   <!-- IMU  -->
   <xacro:default_imu namespace="${namespace}" parent_link="base_link">
@@ -41,6 +38,6 @@
     <origin xyz="0.29 .05 0." rpy="0 0 0"/>
   </xacro:default_camera>
-  <xacro:default_camera namespace="${namespace}" parent_link="base_link" suffix="_under_stereo_right">
-    <origin xyz="0.15 0.10 -0.06" rpy="0 ${0.5*pi} 0"/>
-  </xacro:default_camera>
+  <xacro:stereo_camera namespace="${namespace}" parent_link="base_link" suffix="under">
+    <origin xyz="0.29 0 -0.06" rpy="0 ${0.5*pi} 0"/>
+  </xacro:stereo_camera>
 </robot>

File: uuv-simulator/uuv_sensor_plugins/uuv_sensor_ros_plugins/urdf/stereo_snippets.xacro (robot description, xacro)
@@ -33,5 +33,5 @@
     </collision>
   </xacro:macro>
-  <xacro:macro name="duo3d_camera" params="namespace parent_link *origin">
+  <xacro:macro name="stereo_camera" params="namespace parent_link suffix *origin">
     <link name="duo3d_left_link">
       <inertial>
@@ -78,6 +78,6 @@
         <alwaysOn>true</alwaysOn>
         <updateRate>30.0</updateRate>
-        <cameraName>duo3d_left</cameraName>
-        <imageTopicName>image_raw</imageTopicName>
+        <cameraName>stereo_camera_left_${suffix}</cameraName>
+        <imageTopicName>camera_image</imageTopicName>
         <cameraInfoTopicName>camera_info</cameraInfoTopicName>
         <frameName>duo3d_left_link</frameName>
@@ -133,6 +133,6 @@
         <alwaysOn>true</alwaysOn>
         <updateRate>30.0</updateRate>
-        <cameraName>duo3d_right</cameraName>
-        <imageTopicName>image_raw</imageTopicName>
+        <cameraName>stereo_camera_right_${suffix}</cameraName>
+        <imageTopicName>camera_image</imageTopicName>
         <cameraInfoTopicName>camera_info</cameraInfoTopicName>
         <frameName>duo3d_right_link</frameName>

Commit message: added stereo image proc to forward facing camera as well, stereo vision is pretty jagged but will do

File: tauv_config/albatross_description/urdf/sensors.xacro (robot description, xacro)
@@ -31,13 +31,10 @@
     <origin xyz="0 0 0" rpy="${0} ${0} ${0}"/>
   </xacro:default_imu>
-  <!-- Mount a camera -->
-  <xacro:default_camera namespace="${namespace}" parent_link="base_link" suffix="_front_stereo_left">
+  <!-- Mount cameras -->
+  <xacro:stereo_camera namespace="${namespace}" parent_link="base_link" suffix="under">
+    <origin xyz="0.29 0 -0.06" rpy="0 ${0.5*pi} 0${pi}"/>
+  </xacro:stereo_camera>
+  <xacro:stereo_camera namespace="${namespace}" parent_link="base_link" suffix="front">
     <origin xyz="0.29 -0.10 0." rpy="0 0 0"/>
-  </xacro:default_camera>
-  <xacro:default_camera namespace="${namespace}" parent_link="base_link" suffix="_front_stereo_right">
-    <origin xyz="0.29 .05 0." rpy="0 0 0"/>
-  </xacro:default_camera>
-  <xacro:stereo_camera namespace="${namespace}" parent_link="base_link" suffix="under">
-    <origin xyz="0.29 0 -0.06" rpy="0 ${0.5*pi} 0"/>
   </xacro:stereo_camera>
 </robot>

File: uuv-simulator/uuv_sensor_plugins/uuv_sensor_ros_plugins/urdf/stereo_snippets.xacro (robot description, xacro)
@@ -34,5 +34,5 @@
   </xacro:macro>
   <xacro:macro name="stereo_camera" params="namespace parent_link suffix *origin">
-    <link name="duo3d_left_link">
+    <link name="duo3d_left_link_${suffix}">
       <inertial>
         <mass value="0.01"/>
@@ -46,13 +46,13 @@
       <xacro:no_collision/>
     </link>
-    <joint name="duo3d_joint" type="revolute">
+    <joint name="duo3d_joint_${suffix}" type="revolute">
       <xacro:insert_block name="origin" />
       <parent link="${parent_link}" />
-      <child link="duo3d_left_link" />
+      <child link="duo3d_left_link_${suffix}" />
       <limit upper="0" lower="0" effort="0" velocity="0" />
       <axis xyz="1 0 0"/>
     </joint>
-    <gazebo reference="duo3d_left_link">
-      <sensor name="camera" type="camera">
+    <gazebo reference="duo3d_left_link_${suffix}">
+      <sensor name="camera_${suffix}" type="camera">
       <camera>
         <horizontal_fov>${hfov}</horizontal_fov>
@@ -75,5 +75,5 @@
         </distortion>
       </camera>
-      <plugin name="left_controller" filename="libgazebo_ros_camera.so">
+      <plugin name="left_controller_${suffix}" filename="libgazebo_ros_camera.so">
         <alwaysOn>true</alwaysOn>
         <updateRate>30.0</updateRate>
@@ -94,5 +94,5 @@
     </sensor>
     </gazebo>
-    <link name="duo3d_right_link">
+    <link name="duo3d_right_link_${suffix}">
       <inertial>
         <mass value="0.01"/>
@@ -101,13 +101,13 @@
       <xacro:no_collision/>
     </link>
-    <joint name="duo3d_right_joint" type="revolute">
+    <joint name="duo3d_right_joint_${suffix}" type="revolute">
       <origin xyz="0.0 -0.03 0" rpy="0 0 0"/>
-      <parent link="duo3d_left_link" />
-      <child link="duo3d_right_link" />
+      <parent link="duo3d_left_link_${suffix}" />
+      <child link="duo3d_right_link_${suffix}" />
       <limit upper="0" lower="0" effort="0" velocity="0" />
       <axis xyz="1 0 0"/>
     </joint>
-    <gazebo reference="duo3d_right_link">
-      <sensor name="camera" type="camera">
+    <gazebo reference="duo3d_right_link_${suffix}">
+      <sensor name="camera_${suffix}" type="camera">
       <camera>
         <horizontal_fov>${hfov}</horizontal_fov>
@@ -130,5 +130,5 @@
         </distortion>
       </camera>
-      <plugin name="right_controller" filename="libgazebo_ros_camera.so">
+      <plugin name="right_controller_${suffix}" filename="libgazebo_ros_camera.so">
         <alwaysOn>true</alwaysOn>
         <updateRate>30.0</updateRate>

Commit message: added functions to test the dummy_detector, also archetypes for pixel->depth reprojection

File: tauv_config/albatross_description/urdf/sensors.xacro (robot description, xacro)
@@ -13,5 +13,5 @@
   <!-- Forward-looking sonar sensor -->
   <xacro:forward_multibeam_p900 namespace="${namespace}" parent_link="base_link">
-    <origin xyz="0 0 0" rpy="0 0 0"/>
+    <origin xyz="0 0 0" rpy="0 ${0.5*pi} 0"/>
   </xacro:forward_multibeam_p900>
   <!-- DVL  -->
@@ -35,5 +35,5 @@
     <origin xyz="0.29 0 -0.06" rpy="0 ${0.5*pi} 0${pi}"/>
   </xacro:stereo_camera>
-  <xacro:stereo_camera namespace="${namespace}" parent_link="base_link" suffix="front">
+  <xacro:stereo_camera namespace="" parent_link="base_link" suffix="front">
     <origin xyz="0.29 -0.10 0." rpy="0 0 0"/>
   </xacro:stereo_camera>

File: uuv-simulator/uuv_sensor_plugins/uuv_sensor_ros_plugins/urdf/sonar_snippets.xacro (robot description, xacro)
@@ -142,5 +142,5 @@
       <plugin name="sonar${suffix}_controller" filename="libgazebo_ros_gpu_laser.so">
         <topicName>${topic}</topicName>
-        <frameName>sonar${suffix}_link</frameName>
+        <frameName>/sonar${suffix}_link</frameName>
       </plugin>
       <!-- TODO: Separate switchable sonar version in another macro -->

File: uuv-simulator/uuv_sensor_plugins/uuv_sensor_ros_plugins/urdf/stereo_snippets.xacro (robot description, xacro)
@@ -81,5 +81,5 @@
         <imageTopicName>camera_image</imageTopicName>
         <cameraInfoTopicName>camera_info</cameraInfoTopicName>
-        <frameName>duo3d_left_link</frameName>
+        <frameName>/duo3d_left_link_${suffix}</frameName>
         <hackBaseline>0.07</hackBaseline>
         <distortionK1>${k1l}</distortionK1>
@@ -136,5 +136,5 @@
         <imageTopicName>camera_image</imageTopicName>
         <cameraInfoTopicName>camera_info</cameraInfoTopicName>
-        <frameName>duo3d_right_link</frameName>
+        <frameName>/duo3d_right_link_${suffix}</frameName>
         <hackBaseline>0.07</hackBaseline>
         <distortionK1>${k1l}</distortionK1>

Commit message: explicitly included stereo tuning parameters in yaml file

File: tauv_config/albatross_description/urdf/sensors.xacro (robot description, xacro)
@@ -13,5 +13,5 @@
   <!-- Forward-looking sonar sensor -->
   <xacro:forward_multibeam_p900 namespace="${namespace}" parent_link="base_link">
-    <origin xyz="0 0 0" rpy="0 ${0.5*pi} 0"/>
+    <origin xyz="0 0 0" rpy="0 0 0"/>
   </xacro:forward_multibeam_p900>
   <!-- DVL  -->

Commit message: added yolo and various other slam things

File: tauv_config/albatross_description/urdf/sensors.xacro (robot description, xacro)
@@ -33,8 +33,11 @@
   <!-- Mount cameras -->
   <xacro:stereo_camera namespace="${namespace}" parent_link="base_link" suffix="under">
-    <origin xyz="0.29 0 -0.06" rpy="0 ${0.5*pi} 0${pi}"/>
+    <origin xyz="0.29 0 -0.06" rpy="0 ${0.5*pi} ${pi}"/>
   </xacro:stereo_camera>
   <xacro:stereo_camera namespace="" parent_link="base_link" suffix="front">
-    <origin xyz="0.29 -0.10 0." rpy="0 0 0"/>
+    <origin xyz="0.32 0.0 0.0" rpy="0 0 0"/>
   </xacro:stereo_camera>
+<!--  <xacro:default_camera namespace="" parent_link="base_link" suffix="front">-->
+<!--    <origin xyz="0.32 0.0 0.0" rpy="0 0 0"/>-->
+<!--  </xacro:default_camera>-->
 </robot>

File: uuv-simulator/uuv_sensor_plugins/uuv_sensor_ros_plugins/urdf/stereo_snippets.xacro (robot description, xacro)
@@ -34,4 +34,22 @@
   </xacro:macro>
   <xacro:macro name="stereo_camera" params="namespace parent_link suffix *origin">
+    <link name="duo3d_left_link_stabilized_${suffix}">
+      <inertial>
+        <mass value="0.01"/>
+        <inertia ixx="0.0001" ixy="0" ixz="0" iyy="0.0001" iyz="0" izz="0.0001" />
+      </inertial>
+      <visual>
+        <geometry>
+          <mesh filename="file://$(find uuv_sensor_ros_plugins)/meshes/duo3d.dae"/>
+        </geometry>
+      </visual>
+      <xacro:no_collision/>
+    </link>
+    <joint name="duo3d_stabilized_joint_${suffix}" type="fixed">
+      <xacro:insert_block name="origin" />
+      <preserveFixedJoint>true</preserveFixedJoint>
+      <parent link="${parent_link}"/>
+      <child link="duo3d_left_link_stabilized_${suffix}"/>
+    </joint>
     <link name="duo3d_left_link_${suffix}">
       <inertial>
@@ -39,18 +57,38 @@
         <inertia ixx="0" ixy="0.0" ixz="0.0" iyy="0" iyz="0.0" izz="0" />
       </inertial>
+      <xacro:no_collision/>
+    </link>
+    <joint name="duo3d_joint_${suffix}" type="fixed">
+      <axis xyz="0 0 1"/>
+      <origin xyz="0 0 0" rpy="0 0 0"/>
+      <parent link="duo3d_left_link_stabilized_${suffix}" />
+      <child link="duo3d_left_link_${suffix}" />
+      <limit upper="0" lower="0" effort="0" velocity="0" />
+    </joint>
+    <joint name="duo3d_optical_joint_${suffix}" type="revolute">
+      <origin xyz="0 0 0" rpy="${-pi/2} 0 ${-pi/2}"/>
+      <parent link="duo3d_left_link_${suffix}"/>
+      <child link="duo3d_optical_link_${suffix}"/>
+      <limit upper="0" lower="0" effort="0" velocity="0" />
+      <axis xyz="1 0 0"/>
+    </joint>
+    <link name="duo3d_optical_link_${suffix}">
+      <xacro:box_inertial x="0.0001" y="0.0001" z="0.0001" mass="0.001">
+        <origin xyz="0 0 0" rpy="0 0 0"/>
+      </xacro:box_inertial>
+      <collision>
+        <!-- todo: gazebo needs a collision volume or it will ignore the pose of
+           the joint that leads to this link (and assume it to be the identity) -->
+        <geometry>
+          <cylinder length="0.000001" radius="0.000001"/>
+        </geometry>
+        <origin xyz="0 0 0" rpy="0 ${0.5*pi} 0"/>
+      </collision>
       <visual>
         <geometry>
-          <mesh filename="file://$(find uuv_sensor_ros_plugins)/meshes/duo3d.dae"/>
+          <cylinder length="0.000001" radius="0.000001"/>
         </geometry>
       </visual>
-      <xacro:no_collision/>
-    </link>
-    <joint name="duo3d_joint_${suffix}" type="revolute">
-      <xacro:insert_block name="origin" />
-      <parent link="${parent_link}" />
-      <child link="duo3d_left_link_${suffix}" />
-      <limit upper="0" lower="0" effort="0" velocity="0" />
-      <axis xyz="1 0 0"/>
-    </joint>
+    </link>
     <gazebo reference="duo3d_left_link_${suffix}">
       <sensor name="camera_${suffix}" type="camera">
@@ -81,6 +119,6 @@
         <imageTopicName>camera_image</imageTopicName>
         <cameraInfoTopicName>camera_info</cameraInfoTopicName>
-        <frameName>/duo3d_left_link_${suffix}</frameName>
-        <hackBaseline>0.07</hackBaseline>
+        <frameName>/duo3d_optical_link_${suffix}</frameName>
+        <hackBaseline>0.0</hackBaseline>
         <distortionK1>${k1l}</distortionK1>
         <distortionK2>${k2l}</distortionK2>
@@ -101,11 +139,36 @@
       <xacro:no_collision/>
     </link>
-    <joint name="duo3d_right_joint_${suffix}" type="revolute">
-      <origin xyz="0.0 -0.03 0" rpy="0 0 0"/>
+    <joint name="duo3d_right_joint_${suffix}" type="fixed">
+      <origin xyz="0.0 0.03  0.0" rpy="0 0 0"/>
       <parent link="duo3d_left_link_${suffix}" />
       <child link="duo3d_right_link_${suffix}" />
       <limit upper="0" lower="0" effort="0" velocity="0" />
+      <axis xyz="0 0 1"/>
+    </joint>
+    <joint name="duo3d_optical_joint_right_${suffix}" type="revolute">
+      <origin xyz="0 0 0" rpy="${-pi/2} 0 ${-pi/2}"/>
+      <parent link="duo3d_right_link_${suffix}"/>
+      <child link="duo3d_optical_link_right_${suffix}"/>
+      <limit upper="0" lower="0" effort="0" velocity="0" />
       <axis xyz="1 0 0"/>
     </joint>
+    <link name="duo3d_optical_link_right_${suffix}">
+      <xacro:box_inertial x="0.0001" y="0.0001" z="0.0001" mass="0.001">
+        <origin xyz="0 0 0" rpy="0 0 0"/>
+      </xacro:box_inertial>
+      <collision>
+        <!-- todo: gazebo needs a collision volume or it will ignore the pose of
+           the joint that leads to this link (and assume it to be the identity) -->
+        <geometry>
+          <cylinder length="0.000001" radius="0.000001"/>
+        </geometry>
+        <origin xyz="0 0 0" rpy="0 ${0.5*pi} 0"/>
+      </collision>
+      <visual>
+        <geometry>
+          <cylinder length="0.000001" radius="0.000001"/>
+        </geometry>
+      </visual>
+    </link>
     <gazebo reference="duo3d_right_link_${suffix}">
       <sensor name="camera_${suffix}" type="camera">
@@ -137,5 +200,5 @@
         <cameraInfoTopicName>camera_info</cameraInfoTopicName>
         <frameName>/duo3d_right_link_${suffix}</frameName>
-        <hackBaseline>0.07</hackBaseline>
+        <hackBaseline>0.0</hackBaseline>
         <distortionK1>${k1l}</distortionK1>
         <distortionK2>${k2l}</distortionK2>
