Commit message: unholy gods help me

File: tauv_config/albatross_description/urdf/sensors.xacro (robot description, xacro)
@@ -11,8 +11,8 @@
   <!-- Mount a Pose 3D sensor. -->
   <xacro:default_pose_3d namespace="${namespace}" parent_link="base_link" />
-  <!-- Forward-looking sonar sensor -->
-  <xacro:forward_multibeam_p900 namespace="${namespace}" parent_link="base_link">
-    <origin xyz="0 0 0" rpy="0 0 0"/>
-  </xacro:forward_multibeam_p900>
+<!--  &lt;!&ndash; Forward-looking sonar sensor &ndash;&gt;-->
+<!--  <xacro:forward_multibeam_p900 namespace="${namespace}" parent_link="base_link">-->
+<!--    <origin xyz="0 0 0" rpy="0 0 0"/>-->
+<!--  </xacro:forward_multibeam_p900>-->
   <!-- DVL  -->
   <xacro:default_dvl namespace="${namespace}" parent_link="base_link">
@@ -38,4 +38,7 @@
     <origin xyz="0.32 0.0 0.0" rpy="0 0 0"/>
   </xacro:stereo_camera>
+  <xacro:forward_multibeam_sonar_m450_130 namespace="" parent_link="base_link" suffix="topside">
+    <origin xyz=".32 0.0 .5" rpy="0 0 0"/>
+  </xacro:forward_multibeam_sonar_m450_130 >
 <!--  <xacro:default_camera namespace="" parent_link="base_link" suffix="front">-->
 <!--    <origin xyz="0.32 0.0 0.0" rpy="0 0 0"/>-->

File: uuv-simulator/uuv_sensor_plugins/uuv_sensor_ros_plugins/urdf/sonar_snippets.xacro (robot description, xacro)
@@ -48,12 +48,12 @@
   </xacro:macro>
   <!-- Inspired by m450-130: http://www.blueview.com/products/2d-imaging-sonar/m900-series/ -->
-  <xacro:macro name="forward_multibeam_sonar_m450_130" params="namespace parent_link *origin">
+  <xacro:macro name="forward_multibeam_sonar_m450_130" params="namespace parent_link suffix *origin">
     <xacro:multibeam_sonar
       namespace="${namespace}"
-      suffix=""
+      suffix="${suffix}"
       parent_link="${parent_link}"
       topic="sonar"
       mass="0.015"
-      update_rate="25"
+      update_rate="1/11"
       samples="768"
       fov="2.27"
@@ -116,7 +116,7 @@
   </joint>
   <gazebo reference="sonar${suffix}_link">
-    <sensor type="gpu_ray" name="sonar${suffix}">
+    <sensor type="ray" name="sonar${suffix}">
       <pose>0 0 0 0 0 0</pose>
-      <visualize>false</visualize>
+      <visualize>true</visualize>
       <update_rate>${update_rate}</update_rate>
       <ray>
@@ -140,5 +140,5 @@
         </noise>
       </ray>
-      <plugin name="sonar${suffix}_controller" filename="libgazebo_ros_gpu_laser.so">
+      <plugin name="sonar${suffix}_controller" filename="libgazebo_ros_laser.so">
         <topicName>${topic}</topicName>
         <frameName>/sonar${suffix}_link</frameName>

File: uuv-simulator/uuv_sensor_plugins/uuv_sensor_ros_plugins/urdf/stereo_snippets.xacro (robot description, xacro)
@@ -140,5 +140,5 @@
     </link>
     <joint name="duo3d_right_joint_${suffix}" type="fixed">
-      <origin xyz="0.0 0.03  0.0" rpy="0 0 0"/>
+      <origin xyz="0.0 0.03 0.0" rpy="0 0 0"/>
       <parent link="duo3d_left_link_${suffix}" />
       <child link="duo3d_right_link_${suffix}" />
@@ -199,5 +199,5 @@
         <imageTopicName>camera_image</imageTopicName>
         <cameraInfoTopicName>camera_info</cameraInfoTopicName>
-        <frameName>/duo3d_right_link_${suffix}</frameName>
+        <frameName>/duo3d_optical_link_right_${suffix}</frameName>
         <hackBaseline>0.0</hackBaseline>
         <distortionK1>${k1l}</distortionK1>

Commit message: Advaith/visionbucket (#44)
* changed to not publish false

* imu urdf level

* removing position ekf

* set params in madgwick

* ended base footprint boradcaster

* changed imu urdf

* publishing imu topic as tf now

* set publish roll pitch

* changed topic

* running comp filter

* remove nodelet

* reverted imu pos

* back to madgwick, pub tf

* accel

* moving to ekf

* urdf

* urdf back

* added yaw to imu

* IMU regular now

* ransformter

* dvl testing

* working on bucket

* built bucket messages

* fixing build errors

* fixing build errors

* updated

* fixed weird package error

* ekf is publishing transform again, changed joystick input for teleop controller and joystick works

* added service to register detection against Detection_Bucket

* added vision_msgs to dependencies

* running stereo_image_proc on downward cameras

* undid the pose_gt file changes

* added 3D bbox to bucket_detection message, detector_bucket.py publishes 3d bbox now

* fixed detector __init__.py file, added 3d bounding box to BucketDetection message, detector_bucket publishes BoundingBoxArray

* removed ns=gnc from launch file, added objects to underwater_heightmap world

* removed accidental mod to controller.py

* removed imu_complementary filter dependency, we are using madgwick filter

* added stereo image proc to forward facing camera as well, stereo vision is pretty jagged but will do

* added functions to test the dummy_detector, also archetypes for pixel->depth reprojection

* explicitly included stereo tuning parameters in yaml file

* added pose graph skeleton

* added yolo and various other slam things

* unholy gods help me

* adjustments to PR

* cleanup

* removed depth odom from gnc launch file

* added depth odom into efk_params

File: tauv_config/albatross_description/urdf/sensors.xacro (robot description, xacro)
@@ -11,8 +11,8 @@
   <!-- Mount a Pose 3D sensor. -->
   <xacro:default_pose_3d namespace="${namespace}" parent_link="base_link" />
-  <!-- Forward-looking sonar sensor -->
-  <xacro:forward_multibeam_p900 namespace="${namespace}" parent_link="base_link">
-    <origin xyz="0 0 0" rpy="0 0 0"/>
-  </xacro:forward_multibeam_p900>
+<!--  &lt;!&ndash; Forward-looking sonar sensor &ndash;&gt;-->
+<!--  <xacro:forward_multibeam_p900 namespace="${namespace}" parent_link="base_link">-->
+<!--    <origin xyz="0 0 0" rpy="0 0 0"/>-->
+<!--  </xacro:forward_multibeam_p900>-->
   <!-- DVL  -->
   <xacro:default_dvl namespace="${namespace}" parent_link="base_link">
@@ -27,17 +27,20 @@
     <origin xyz="0 0 0" rpy="0 0 0"/>
   </xacro:default_pressure>
-  <xacro:default_camera namespace="${namespace}" parent_link="base_link" suffix="under2">
-    <origin xyz="0.15 -0.05 -0.06" rpy="0 ${0.5*pi} 0"/>
-  </xacro:default_camera>
   <!-- IMU  -->
   <xacro:default_imu namespace="${namespace}" parent_link="base_link">
     <origin xyz="0 0 0" rpy="${0} ${0} ${0}"/>
   </xacro:default_imu>
-  <!-- Mount a camera -->
-  <xacro:default_camera namespace="${namespace}" parent_link="base_link" suffix="front">
-    <origin xyz="0.29 0.0 0." rpy="0 0 0"/>
-  </xacro:default_camera>
-  <xacro:default_camera namespace="${namespace}" parent_link="base_link" suffix="under1">
-    <origin xyz="0.15 0.05 -0.06" rpy="0 ${0.5*pi} 0"/>
-  </xacro:default_camera>
+  <!-- Mount cameras -->
+  <xacro:stereo_camera namespace="${namespace}" parent_link="base_link" suffix="under">
+    <origin xyz="0.29 0 -0.06" rpy="0 ${0.5*pi} ${pi}"/>
+  </xacro:stereo_camera>
+  <xacro:stereo_camera namespace="" parent_link="base_link" suffix="front">
+    <origin xyz="0.32 0.0 0.0" rpy="0 0 0"/>
+  </xacro:stereo_camera>
+  <xacro:forward_multibeam_sonar_m450_130 namespace="" parent_link="base_link" suffix="topside">
+    <origin xyz=".32 0.0 .5" rpy="0 0 0"/>
+  </xacro:forward_multibeam_sonar_m450_130 >
+<!--  <xacro:default_camera namespace="" parent_link="base_link" suffix="front">-->
+<!--    <origin xyz="0.32 0.0 0.0" rpy="0 0 0"/>-->
+<!--  </xacro:default_camera>-->
 </robot>

File: uuv-simulator/uuv_sensor_plugins/uuv_sensor_ros_plugins/urdf/sonar_snippets.xacro (robot description, xacro)
@@ -48,12 +48,12 @@
   </xacro:macro>
   <!-- Inspired by m450-130: http://www.blueview.com/products/2d-imaging-sonar/m900-series/ -->
-  <xacro:macro name="forward_multibeam_sonar_m450_130" params="namespace parent_link *origin">
+  <xacro:macro name="forward_multibeam_sonar_m450_130" params="namespace parent_link suffix *origin">
     <xacro:multibeam_sonar
       namespace="${namespace}"
-      suffix=""
+      suffix="${suffix}"
       parent_link="${parent_link}"
       topic="sonar"
       mass="0.015"
-      update_rate="25"
+      update_rate="1/11"
       samples="768"
       fov="2.27"
@@ -116,7 +116,7 @@
   </joint>
   <gazebo reference="sonar${suffix}_link">
-    <sensor type="gpu_ray" name="sonar${suffix}">
+    <sensor type="ray" name="sonar${suffix}">
       <pose>0 0 0 0 0 0</pose>
-      <visualize>false</visualize>
+      <visualize>true</visualize>
       <update_rate>${update_rate}</update_rate>
       <ray>
@@ -140,7 +140,7 @@
         </noise>
       </ray>
-      <plugin name="sonar${suffix}_controller" filename="libgazebo_ros_gpu_laser.so">
+      <plugin name="sonar${suffix}_controller" filename="libgazebo_ros_laser.so">
         <topicName>${topic}</topicName>
-        <frameName>sonar${suffix}_link</frameName>
+        <frameName>/sonar${suffix}_link</frameName>
       </plugin>
       <!-- TODO: Separate switchable sonar version in another macro -->

File: uuv-simulator/uuv_sensor_plugins/uuv_sensor_ros_plugins/urdf/stereo_snippets.xacro (robot description, xacro)
@@ -33,26 +33,64 @@
     </collision>
   </xacro:macro>
-  <xacro:macro name="duo3d_camera" params="namespace parent_link *origin">
-    <link name="duo3d_left_link">
+  <xacro:macro name="stereo_camera" params="namespace parent_link suffix *origin">
+    <link name="duo3d_left_link_stabilized_${suffix}">
+      <inertial>
+        <mass value="0.01"/>
+        <inertia ixx="0.0001" ixy="0" ixz="0" iyy="0.0001" iyz="0" izz="0.0001" />
+      </inertial>
+      <visual>
+        <geometry>
+          <mesh filename="file://$(find uuv_sensor_ros_plugins)/meshes/duo3d.dae"/>
+        </geometry>
+      </visual>
+      <xacro:no_collision/>
+    </link>
+    <joint name="duo3d_stabilized_joint_${suffix}" type="fixed">
+      <xacro:insert_block name="origin" />
+      <preserveFixedJoint>true</preserveFixedJoint>
+      <parent link="${parent_link}"/>
+      <child link="duo3d_left_link_stabilized_${suffix}"/>
+    </joint>
+    <link name="duo3d_left_link_${suffix}">
       <inertial>
         <mass value="0.01"/>
         <inertia ixx="0" ixy="0.0" ixz="0.0" iyy="0" iyz="0.0" izz="0" />
       </inertial>
+      <xacro:no_collision/>
+    </link>
+    <joint name="duo3d_joint_${suffix}" type="fixed">
+      <axis xyz="0 0 1"/>
+      <origin xyz="0 0 0" rpy="0 0 0"/>
+      <parent link="duo3d_left_link_stabilized_${suffix}" />
+      <child link="duo3d_left_link_${suffix}" />
+      <limit upper="0" lower="0" effort="0" velocity="0" />
+    </joint>
+    <joint name="duo3d_optical_joint_${suffix}" type="revolute">
+      <origin xyz="0 0 0" rpy="${-pi/2} 0 ${-pi/2}"/>
+      <parent link="duo3d_left_link_${suffix}"/>
+      <child link="duo3d_optical_link_${suffix}"/>
+      <limit upper="0" lower="0" effort="0" velocity="0" />
+      <axis xyz="1 0 0"/>
+    </joint>
+    <link name="duo3d_optical_link_${suffix}">
+      <xacro:box_inertial x="0.0001" y="0.0001" z="0.0001" mass="0.001">
+        <origin xyz="0 0 0" rpy="0 0 0"/>
+      </xacro:box_inertial>
+      <collision>
+        <!-- todo: gazebo needs a collision volume or it will ignore the pose of
+           the joint that leads to this link (and assume it to be the identity) -->
+        <geometry>
+          <cylinder length="0.000001" radius="0.000001"/>
+        </geometry>
+        <origin xyz="0 0 0" rpy="0 ${0.5*pi} 0"/>
+      </collision>
       <visual>
         <geometry>
-          <mesh filename="file://$(find uuv_sensor_ros_plugins)/meshes/duo3d.dae"/>
+          <cylinder length="0.000001" radius="0.000001"/>
         </geometry>
       </visual>
-      <xacro:no_collision/>
-    </link>
-    <joint name="duo3d_joint" type="revolute">
-      <xacro:insert_block name="origin" />
-      <parent link="${parent_link}" />
-      <child link="duo3d_left_link" />
-      <limit upper="0" lower="0" effort="0" velocity="0" />
-      <axis xyz="1 0 0"/>
-    </joint>
-    <gazebo reference="duo3d_left_link">
-      <sensor name="camera" type="camera">
+    </link>
+    <gazebo reference="duo3d_left_link_${suffix}">
+      <sensor name="camera_${suffix}" type="camera">
       <camera>
         <horizontal_fov>${hfov}</horizontal_fov>
@@ -75,12 +113,12 @@
         </distortion>
       </camera>
-      <plugin name="left_controller" filename="libgazebo_ros_camera.so">
+      <plugin name="left_controller_${suffix}" filename="libgazebo_ros_camera.so">
         <alwaysOn>true</alwaysOn>
         <updateRate>30.0</updateRate>
-        <cameraName>duo3d_left</cameraName>
-        <imageTopicName>image_raw</imageTopicName>
+        <cameraName>stereo_camera_left_${suffix}</cameraName>
+        <imageTopicName>camera_image</imageTopicName>
         <cameraInfoTopicName>camera_info</cameraInfoTopicName>
-        <frameName>duo3d_left_link</frameName>
-        <hackBaseline>0.07</hackBaseline>
+        <frameName>/duo3d_optical_link_${suffix}</frameName>
+        <hackBaseline>0.0</hackBaseline>
         <distortionK1>${k1l}</distortionK1>
         <distortionK2>${k2l}</distortionK2>
@@ -94,5 +132,5 @@
     </sensor>
     </gazebo>
-    <link name="duo3d_right_link">
+    <link name="duo3d_right_link_${suffix}">
       <inertial>
         <mass value="0.01"/>
@@ -101,13 +139,38 @@
       <xacro:no_collision/>
     </link>
-    <joint name="duo3d_right_joint" type="revolute">
-      <origin xyz="0.0 -0.03 0" rpy="0 0 0"/>
-      <parent link="duo3d_left_link" />
-      <child link="duo3d_right_link" />
+    <joint name="duo3d_right_joint_${suffix}" type="fixed">
+      <origin xyz="0.0 0.03 0.0" rpy="0 0 0"/>
+      <parent link="duo3d_left_link_${suffix}" />
+      <child link="duo3d_right_link_${suffix}" />
+      <limit upper="0" lower="0" effort="0" velocity="0" />
+      <axis xyz="0 0 1"/>
+    </joint>
+    <joint name="duo3d_optical_joint_right_${suffix}" type="revolute">
+      <origin xyz="0 0 0" rpy="${-pi/2} 0 ${-pi/2}"/>
+      <parent link="duo3d_right_link_${suffix}"/>
+      <child link="duo3d_optical_link_right_${suffix}"/>
       <limit upper="0" lower="0" effort="0" velocity="0" />
       <axis xyz="1 0 0"/>
     </joint>
-    <gazebo reference="duo3d_right_link">
-      <sensor name="camera" type="camera">
+    <link name="duo3d_optical_link_right_${suffix}">
+      <xacro:box_inertial x="0.0001" y="0.0001" z="0.0001" mass="0.001">
+        <origin xyz="0 0 0" rpy="0 0 0"/>
+      </xacro:box_inertial>
+      <collision>
+        <!-- todo: gazebo needs a collision volume or it will ignore the pose of
+           the joint that leads to this link (and assume it to be the identity) -->
+        <geometry>
+          <cylinder length="0.000001" radius="0.000001"/>
+        </geometry>
+        <origin xyz="0 0 0" rpy="0 ${0.5*pi} 0"/>
+      </collision>
+      <visual>
+        <geometry>
+          <cylinder length="0.000001" radius="0.000001"/>
+        </geometry>
+      </visual>
+    </link>
+    <gazebo reference="duo3d_right_link_${suffix}">
+      <sensor name="camera_${suffix}" type="camera">
       <camera>
         <horizontal_fov>${hfov}</horizontal_fov>
@@ -130,12 +193,12 @@
         </distortion>
       </camera>
-      <plugin name="right_controller" filename="libgazebo_ros_camera.so">
+      <plugin name="right_controller_${suffix}" filename="libgazebo_ros_camera.so">
         <alwaysOn>true</alwaysOn>
         <updateRate>30.0</updateRate>
-        <cameraName>duo3d_right</cameraName>
-        <imageTopicName>image_raw</imageTopicName>
+        <cameraName>stereo_camera_right_${suffix}</cameraName>
+        <imageTopicName>camera_image</imageTopicName>
         <cameraInfoTopicName>camera_info</cameraInfoTopicName>
-        <frameName>duo3d_right_link</frameName>
-        <hackBaseline>0.07</hackBaseline>
+        <frameName>/duo3d_optical_link_right_${suffix}</frameName>
+        <hackBaseline>0.0</hackBaseline>
         <distortionK1>${k1l}</distortionK1>
         <distortionK2>${k2l}</distortionK2>
