Commit message: fix uuv snippets causing gazebo crashes

File: uuv-simulator/uuv_sensor_plugins/uuv_sensor_ros_plugins/urdf/camera_snippets.xacro (robot description, xacro)
@@ -93,4 +93,9 @@
         <origin xyz="0 0 0" rpy="0 ${0.5*pi} 0"/>
       </collision>
+      <visual>
+        <geometry>
+          <cylinder length="0.000001" radius="0.000001"/>
+        </geometry>
+      </visual>
     </link>
     <joint name="${namespace}/camera${suffix}_optical_joint" type="revolute">

File: uuv-simulator/uuv_sensor_plugins/uuv_sensor_ros_plugins/urdf/imu_snippets.xacro (robot description, xacro)
@@ -124,9 +124,13 @@
     <!-- IMU link -->
     <link name="${namespace}/imu${imu_suffix}_link">
-      <inertial>
-        <xacro:insert_block name="inertia" />
-        <mass value="${mass_imu_sensor}" />  <!-- [kg] -->
-        <origin xyz="0 0 0" rpy="0 0 0" />
-      </inertial>
+      <xacro:box_inertial x="0.0001" y="0.0001" z="0.0001" mass="${mass_imu_sensor}">
+        <origin xyz="0 0 0" rpy="0 0 0"/>
+      </xacro:box_inertial>
+      <xacro:no_collision/>
+      <visual>
+        <geometry>
+          <cylinder length="0.000001" radius="0.000001"/>
+        </geometry>
+      </visual>
     </link>
     <!-- IMU joint -->
