Commit message: fix more uuv links, test frame transforms

File: uuv-simulator/uuv_sensor_plugins/uuv_sensor_ros_plugins/urdf/gps_sensor_snippets.xacro (robot description, xacro)
@@ -24,4 +24,9 @@
          <origin xyz="0 0 0" rpy="0 0 0" />
        </inertial>
+       <visual>
+         <geometry>
+           <box size="0.05 0.05 0.05" />
+         </geometry>
+       </visual>
      </link>
      <!-- GPS joint -->

File: uuv-simulator/uuv_sensor_plugins/uuv_sensor_ros_plugins/urdf/pose_3d_snippets.xacro (robot description, xacro)
@@ -22,4 +22,9 @@
         <origin xyz="0 0 0" rpy="0 0 0" />
       </inertial>
+      <visual>
+        <geometry>
+          <box size="0.05 0.05 0.05" />
+        </geometry>
+      </visual>
     </link>
     <joint name="${namespace}/pose_sensor_${suffix}_joint" type="revolute">
