Commit message: trying to fix test errors with tam

File: tauv_config/manta_description/urdf/manta_base.xacro (robot description, xacro)
@@ -51,5 +51,5 @@
   <xacro:macro name="manta_base" params="namespace *gazebo inertial_reference_frame">
    <!-- Rigid body description of the base link -->
-    <link name="${namespace}/base_link">
+    <link name="base_link">
         <!--
           Be careful to setup the coefficients for the inertial tensor,
@@ -82,5 +82,5 @@
     </collision>
   </link>
-    <gazebo reference="${namespace}/base_link">
+    <gazebo reference="base_link">
       <selfCollide>false</selfCollide>
     </gazebo>

File: tauv_config/manta_description/urdf/manta_gazebo.xacro (robot description, xacro)
@@ -7,5 +7,5 @@
   <xacro:macro name="manta_hydro_model" params="namespace">
     <!-- List of hydrodynamic models this robot's links -->
-    <link name="${namespace}/base_link">
+    <link name="base_link">
       <!-- This flag will make the link neutrally buoyant -->
       <neutrally_buoyant>0</neutrally_buoyant>

File: tauv_config/manta_description/urdf/manta_sensors.xacro (robot description, xacro)
@@ -8,17 +8,17 @@
   <xacro:default_dvl_macro
     namespace="${namespace}"
-    parent_link="${namespace}/base_link"
+    parent_link="base_link"
     inertial_reference_frame="${inertial_reference_frame}">
     <origin xyz="0 0 0" rpy="0 ${0.5*pi} 0"/>
   </xacro:default_dvl_macro>
   <!-- Magnetometer  -->
-  <xacro:default_magnetometer namespace="${namespace}" parent_link="${namespace}/base_link"/>
+  <xacro:default_magnetometer namespace="${namespace}" parent_link="base_link"/>
 <!--
   <!- RPT   ->
-  <xacro:default_rpt namespace="${namespace}" parent_link="${namespace}/base_link">
+  <xacro:default_rpt namespace="${namespace}" parent_link="base_link">
     <origin xyz="-1.32 0 0.8" rpy="0 0 0"/>
   </xacro:default_rpt> -->
   <!-- Pressure  -->
-  <xacro:default_pressure_macro namespace="${namespace}" parent_link="${namespace}/base_link">
+  <xacro:default_pressure_macro namespace="${namespace}" parent_link="base_link">
     <origin xyz="0 0 0" rpy="0 0 0"/>
   </xacro:default_pressure_macro>
@@ -26,25 +26,25 @@
   <xacro:default_imu_macro
     namespace="${namespace}"
-    parent_link="${namespace}/base_link"
+    parent_link="base_link"
     inertial_reference_frame="${inertial_reference_frame}">
     <origin xyz="0 0 0" rpy="0 0 0"/>
   </xacro:default_imu_macro>
   <!-- Mount a camera -->
-  <xacro:default_camera namespace="${namespace}" parent_link="${namespace}/base_link" suffix="front">
+  <xacro:default_camera namespace="${namespace}" parent_link="base_link" suffix="front">
     <origin xyz="0.29 0.0 0." rpy="0 0 0"/>
   </xacro:default_camera>
-  <xacro:default_camera namespace="${namespace}" parent_link="${namespace}/base_link" suffix="under">
+  <xacro:default_camera namespace="${namespace}" parent_link="base_link" suffix="under">
     <origin xyz="0.15 0.0 -0.06" rpy="0 ${0.5*pi} 0"/>
   </xacro:default_camera>
 <!--
-  <xacro:default_camera namespace="${namespace}" parent_link="${namespace}/base_link" suffix="left">
+  <xacro:default_camera namespace="${namespace}" parent_link="base_link" suffix="left">
     <origin xyz="1.15 0.63 0.4" rpy="0 0.6 -0.4"/>
   </xacro:default_camera>   -->
   <!-- Mount a GPS.
-  <xacro:default_gps namespace="${namespace}" parent_link="${namespace}/base_link" /> -->
+  <xacro:default_gps namespace="${namespace}" parent_link="base_link" /> -->
   <!-- Mount a Pose 3D sensor. This will give 3D pose -->
   <xacro:default_pose_3d_macro
     namespace="${namespace}"
-    parent_link="${namespace}/base_link"
+    parent_link="base_link"
     inertial_reference_frame="${inertial_reference_frame}" />
 </robot>
