Commit message: update unit tests with new link names

File: uuv-simulator/uuv_gazebo_plugins/uuv_gazebo_ros_plugins/test/models/default_fossen_vehicle/model.xacro (robot description, xacro)
@@ -13,5 +13,5 @@
 -->
 <robot name="rexrov" xmlns:xacro="http://www.ros.org/wiki/xacro" >
-  <link name="vehicle/base_link">
+  <link name="base_link">
     <inertial>
       <mass value="10"/>
@@ -25,5 +25,5 @@
       <flow_velocity_topic>hydrodynamics/current_velocity</flow_velocity_topic>
       <debug>0</debug>
-      <link name="vehicle/base_link">
+      <link name="base_link">
           <neutrally_buoyant>0</neutrally_buoyant>
           <volume>1.0</volume>

File: uuv-simulator/uuv_gazebo_plugins/uuv_gazebo_ros_plugins/test/models/sphere_vehicle/model.xacro (robot description, xacro)
@@ -13,5 +13,5 @@
 -->
 <robot name="rexrov" xmlns:xacro="http://www.ros.org/wiki/xacro" >
-  <link name="vehicle/base_link">
+  <link name="base_link">
     <inertial>
       <mass value="10"/>
@@ -25,5 +25,5 @@
       <flow_velocity_topic>hydrodynamics/current_velocity</flow_velocity_topic>
       <debug>0</debug>
-      <link name="vehicle/base_link">
+      <link name="base_link">
           <neutrally_buoyant>0</neutrally_buoyant>
           <volume>0.009727626</volume>

File: uuv-simulator/uuv_gazebo_plugins/uuv_gazebo_ros_plugins/test/models/thrusters/model.xacro (robot description, xacro)
@@ -16,5 +16,5 @@
   <xacro:include filename="$(find uuv_gazebo_ros_plugins)/urdf/thruster_snippets.xacro"/>
   <xacro:property name="prop_mesh_file" value="file://$(find uuv_descriptions)/models/rexrov/mesh/prop.dae"/>
-  <link name="vehicle/base_link">
+  <link name="base_link">
     <inertial>
       <mass value="10"/>
@@ -28,5 +28,5 @@
       <flow_velocity_topic>hydrodynamics/current_velocity</flow_velocity_topic>
       <debug>0</debug>
-      <link name="vehicle/base_link">
+      <link name="base_link">
           <neutrally_buoyant>0</neutrally_buoyant>
           <volume>0.009727626</volume>
