Commit message: added temporary swim through gate feature

File: tauv_config/kingfisher_description/urdf/sensors.xacro (robot description, xacro)
@@ -38,7 +38,7 @@
     <origin xyz="0.32 0.0 0.0" rpy="0 0 0"/>
   </xacro:stereo_camera>
-  <xacro:forward_multibeam_sonar_m450_130 namespace="" parent_link="base_link" suffix="topside">
-    <origin xyz=".32 0.0 .5" rpy="0 0 0"/>
-  </xacro:forward_multibeam_sonar_m450_130 >
+<!--  <xacro:forward_multibeam_sonar_m450_130 namespace="" parent_link="base_link" suffix="topside">-->
+<!--    <origin xyz=".32 0.0 .5" rpy="0 0 0"/>-->
+<!--  </xacro:forward_multibeam_sonar_m450_130 >-->
 <!--  <xacro:default_camera namespace="" parent_link="base_link" suffix="front">-->
 <!--    <origin xyz="0.32 0.0 0.0" rpy="0 0 0"/>-->
