Commit message: added some new robot models

File: tauv_config/kingfisher_description/urdf/base.xacro (robot description, xacro)
@@ -23,9 +23,9 @@
     Open the meshes for the RexROV vehicle in Blender to see an example on the mesh placement.
   -->
-  <xacro:property name="visual_mesh_file" value="file://$(find kingfisher_description)/meshes/vehicle.dae"/>
+  <xacro:property name="visual_mesh_file" value="file://$(find kingfisher_description)/meshes/pls.dae"/>
   <!-- Collision geometry mesh, usually in STL format (it is recommended to keep
   this geometry as simple as possible to improve the performance the physics engine
   regarding the computation of collision forces) -->
-  <xacro:property name="collision_mesh_file" value="file://$(find kingfisher_description)/meshes/vehicle.dae"/>
+  <xacro:property name="collision_mesh_file" value="file://$(find kingfisher_description)/meshes/pls.dae"/>
   <!-- Vehicle macro -->
   <xacro:macro name="kingfisher_base" params="namespace *gazebo">

File: tauv_config/kingfisher_description/urdf/gazebo.xacro (robot description, xacro)
@@ -6,5 +6,5 @@
     <xacro:property name="kingfisher_volume" value="0.016"/>
     <!-- Describing the dimensions of the vehicle's bounding box -->
-    <xacro:property name="kingfisher_length" value="1"/>
+    <xacro:property name="kingfisher_length" value="5"/>
     <xacro:property name="kingfisher_width"  value="1"/>
     <xacro:property name="kingfisher_height" value="1"/>

Commit message: added new kingfisher model

File: tauv_config/kingfisher_description/urdf/base.xacro (robot description, xacro)
@@ -23,9 +23,9 @@
     Open the meshes for the RexROV vehicle in Blender to see an example on the mesh placement.
   -->
-  <xacro:property name="visual_mesh_file" value="file://$(find kingfisher_description)/meshes/pls.dae"/>
+  <xacro:property name="visual_mesh_file" value="file://$(find kingfisher_description)/meshes/kingfisher.dae"/>
   <!-- Collision geometry mesh, usually in STL format (it is recommended to keep
   this geometry as simple as possible to improve the performance the physics engine
   regarding the computation of collision forces) -->
-  <xacro:property name="collision_mesh_file" value="file://$(find kingfisher_description)/meshes/pls.dae"/>
+  <xacro:property name="collision_mesh_file" value="file://$(find kingfisher_description)/meshes/kingfisher.dae"/>
   <!-- Vehicle macro -->
   <xacro:macro name="kingfisher_base" params="namespace *gazebo">

File: tauv_config/kingfisher_description/urdf/sensors.xacro (robot description, xacro)
@@ -33,8 +33,8 @@
   <!-- Mount cameras -->
   <xacro:stereo_camera namespace="${namespace}" parent_link="base_link" suffix="under">
-    <origin xyz="0.29 0 -0.06" rpy="0 ${0.5*pi} ${pi}"/>
+    <origin xyz="0.29 0 -0.2" rpy="0 ${0.5*pi} ${pi}"/>
   </xacro:stereo_camera>
   <xacro:stereo_camera namespace="" parent_link="base_link" suffix="front">
-    <origin xyz="0.32 0.0 0.0" rpy="0 0 0"/>
+    <origin xyz="0.45 0.0 0.0" rpy="0 0 0"/>
   </xacro:stereo_camera>
 <!--  <xacro:forward_multibeam_sonar_m450_130 namespace="" parent_link="base_link" suffix="topside">-->

File: uuv-simulator/uuv_sensor_plugins/uuv_sensor_ros_plugins/urdf/dvl_snippets.xacro (robot description, xacro)
@@ -131,9 +131,9 @@
         <inertia ixx="0.000000017" ixy="0" ixz="0" iyy="0.000000017" iyz="0" izz="0.000000017" />
       </inertial>
-      <visual>
-        <geometry>
-          <mesh filename="file://$(find uuv_sensor_ros_plugins)/meshes/dvl.dae" scale="${scale} ${scale} ${scale}"/>
-        </geometry>
-      </visual>
+<!--      <visual>-->
+<!--        <geometry>-->
+<!--          <mesh filename="file://$(find uuv_sensor_ros_plugins)/meshes/dvl.dae" scale="${scale} ${scale} ${scale}"/>-->
+<!--        </geometry>-->
+<!--      </visual>-->
       <xacro:no_collision/>
     </link>
