Commit message: work on migration

File: src/packages/tauv_config/albatross_description/urdf/base.xacro (robot description, xacro)
@@ -2,5 +2,5 @@
 <robot xmlns:xacro="http://www.ros.org/wiki/xacro">
   <!-- Loading some constants -->
-  <xacro:include filename="$(find uuv_descriptions)/models/common/urdf/common.urdf.xacro"/>
+  <xacro:include filename="$(find uuv_descriptions)/urdf/common.urdf.xacro"/>
   <!-- Loading file with sensor macros -->
   <xacro:include filename="$(find uuv_sensor_ros_plugins)/urdf/sensor_snippets.xacro"/>

File: src/packages/tauv_config/albatross_description/urdf/sensors.xacro (robot description, xacro)
@@ -35,8 +35,8 @@
     <origin xyz="0.29 0 -0.06" rpy="0 ${0.5*pi} ${pi}"/>
   </xacro:stereo_camera>
-  <xacro:stereo_camera namespace="" parent_link="base_link" suffix="front">
+  <xacro:stereo_camera namespace="${namespace}" parent_link="base_link" suffix="front">
     <origin xyz="0.32 0.0 0.0" rpy="0 0 0"/>
   </xacro:stereo_camera>
-  <xacro:forward_multibeam_sonar_m450_130 namespace="" parent_link="base_link" suffix="topside">
+  <xacro:forward_multibeam_sonar_m450_130 namespace="${namespace}" parent_link="base_link" suffix="topside">
     <origin xyz=".32 0.0 .5" rpy="0 0 0"/>
   </xacro:forward_multibeam_sonar_m450_130 >

File: src/packages/uuv-simulator/uuv_gazebo_plugins/uuv_gazebo_ros_plugins/urdf/thruster_snippets.xacro (robot description, xacro)
@@ -79,5 +79,5 @@
       <xacro:insert_block name="origin"/>
       <axis xyz="1 0 0"/>
-      <parent link="${namespace}/base_link"/>
+      <parent link="base_link"/>
       <child link="${namespace}/thruster_${thruster_id}"/>
     </joint>

File: src/packages/uuv-simulator/uuv_sensor_plugins/uuv_sensor_ros_plugins/urdf/sonar_snippets.xacro (robot description, xacro)
@@ -108,47 +108,47 @@
       <xacro:no_collision/>
     </link>
-  <joint name="${namespace}_sonar${suffix}_joint" type="revolute">
-    <xacro:insert_block name="origin" />
-    <parent link="${parent_link}" />
-    <child link="sonar${suffix}_link" />
-    <limit upper="0" lower="0" effort="0" velocity="0" />
-    <axis xyz="1 0 0"/>
-  </joint>
-  <gazebo reference="sonar${suffix}_link">
-    <sensor type="ray" name="sonar${suffix}">
-      <pose>0 0 0 0 0 0</pose>
-      <visualize>true</visualize>
-      <update_rate>${update_rate}</update_rate>
-      <ray>
-        <scan>
-          <horizontal>
-            <samples>${samples}</samples>
-            <resolution>1</resolution>
-            <min_angle>-${0.5*fov}</min_angle>
-            <max_angle>${0.5*fov}</max_angle>
-          </horizontal>
-        </scan>
-        <range>
-          <min>${range_min}</min>
-          <max>${range_max}</max>
-          <resolution>0.01</resolution>
-        </range>
-        <noise>
-          <type>gaussian</type>
-          <mean>0.0</mean>
-          <stddev>${range_stddev}</stddev>
-        </noise>
-      </ray>
-      <plugin name="sonar${suffix}_controller" filename="libgazebo_ros_laser.so">
-        <topicName>${topic}</topicName>
-        <frameName>/sonar${suffix}_link</frameName>
-      </plugin>
-      <!-- TODO: Separate switchable sonar version in another macro -->
-      <!-- <plugin name="switchable_sonar{suffix}_ros_interface" filename="libuuv_gazebo_ros_switchable_gpu_ray_sensor.so">
-          <namespace>${namespace}</namespace>
-          <input_topic>${topic}</input_topic>
-      </plugin> -->
-    </sensor>
-  </gazebo>
+    <joint name="${namespace}_sonar${suffix}_joint" type="revolute">
+      <xacro:insert_block name="origin" />
+      <parent link="${parent_link}" />
+      <child link="sonar${suffix}_link" />
+      <limit upper="0" lower="0" effort="0" velocity="0" />
+      <axis xyz="1 0 0"/>
+    </joint>
+    <gazebo reference="sonar${suffix}_link">
+      <sensor type="ray" name="sonar${suffix}">
+        <pose>0 0 0 0 0 0</pose>
+        <visualize>true</visualize>
+        <update_rate>${update_rate}</update_rate>
+        <ray>
+          <scan>
+            <horizontal>
+              <samples>${samples}</samples>
+              <resolution>1</resolution>
+              <min_angle>-${0.5*fov}</min_angle>
+              <max_angle>${0.5*fov}</max_angle>
+            </horizontal>
+          </scan>
+          <range>
+            <min>${range_min}</min>
+            <max>${range_max}</max>
+            <resolution>0.01</resolution>
+          </range>
+          <noise>
+            <type>gaussian</type>
+            <mean>0.0</mean>
+            <stddev>${range_stddev}</stddev>
+          </noise>
+        </ray>
+        <plugin name="sonar${suffix}_controller" filename="libgazebo_ros_laser.so">
+          <topicName>${topic}</topicName>
+          <frameName>/sonar${suffix}_link</frameName>
+        </plugin>
+        <!-- TODO: Separate switchable sonar version in another macro -->
+        <!-- <plugin name="switchable_sonar{suffix}_ros_interface" filename="libuuv_gazebo_ros_switchable_gpu_ray_sensor.so">
+            <namespace>${namespace}</namespace>
+            <input_topic>${topic}</input_topic>
+        </plugin> -->
+      </sensor>
+    </gazebo>
   </xacro:macro>
 </robot>
