Commit message: fix frame errors maybe?

File: src/packages/tauv_config/albatross_description/urdf/sensors.xacro (robot description, xacro)
@@ -38,7 +38,7 @@
     <origin xyz="0.32 0.0 0.0" rpy="0 0 0"/>
   </xacro:stereo_camera>
-  <xacro:forward_multibeam_sonar_m450_130 namespace="${namespace}" parent_link="base_link" suffix="topside">
+  <!-- <xacro:forward_multibeam_sonar_m450_130 namespace="${namespace}" parent_link="base_link" suffix="topside">
     <origin xyz=".32 0.0 .5" rpy="0 0 0"/>
-  </xacro:forward_multibeam_sonar_m450_130 >
+  </xacro:forward_multibeam_sonar_m450_130 > -->
 <!--  <xacro:default_camera namespace="" parent_link="base_link" suffix="front">-->
 <!--    <origin xyz="0.32 0.0 0.0" rpy="0 0 0"/>-->

File: src/packages/uuv-simulator/uuv_gazebo_plugins/uuv_gazebo_ros_plugins/urdf/thruster_snippets.xacro (robot description, xacro)
@@ -76,11 +76,11 @@
             *dynamics
             *conversion">
-    <joint name="${namespace}/thruster_${thruster_id}_joint" type="continuous">
+    <joint name="thruster_${thruster_id}_joint" type="continuous">
       <xacro:insert_block name="origin"/>
       <axis xyz="1 0 0"/>
       <parent link="base_link"/>
-      <child link="${namespace}/thruster_${thruster_id}"/>
+      <child link="thruster_${thruster_id}"/>
     </joint>
-    <link name="${namespace}/thruster_${thruster_id}">
+    <link name="thruster_${thruster_id}">
       <xacro:box_inertial x="0" y="0" z="0" mass="0.001">
         <origin xyz="0 0 0" rpy="0 0 0"/>
@@ -102,7 +102,7 @@
     </link>
     <gazebo>
-      <plugin name="${namespace}_${thruster_id}_thruster_model" filename="libuuv_thruster_ros_plugin.so">
-        <linkName>${namespace}/thruster_${thruster_id}</linkName>
-        <jointName>${namespace}/thruster_${thruster_id}_joint</jointName>
+      <plugin name="${thruster_id}_thruster_model" filename="libuuv_thruster_ros_plugin.so">
+        <linkName>thruster_${thruster_id}</linkName>
+        <jointName>thruster_${thruster_id}_joint</jointName>
         <thrusterID>${thruster_id}</thrusterID>
         <xacro:insert_block name="dynamics"/>
@@ -110,5 +110,5 @@
       </plugin>
     </gazebo>
-    <gazebo reference="${namespace}/thruster_${thruster_id}">
+    <gazebo reference="hruster_${thruster_id}">
       <selfCollide>false</selfCollide>
     </gazebo>

File: src/packages/uuv-simulator/uuv_sensor_plugins/uuv_sensor_ros_plugins/urdf/sonar_snippets.xacro (robot description, xacro)
@@ -108,47 +108,47 @@
       <xacro:no_collision/>
     </link>
-    <joint name="${namespace}_sonar${suffix}_joint" type="revolute">
-      <xacro:insert_block name="origin" />
-      <parent link="${parent_link}" />
-      <child link="sonar${suffix}_link" />
-      <limit upper="0" lower="0" effort="0" velocity="0" />
-      <axis xyz="1 0 0"/>
-    </joint>
-    <gazebo reference="sonar${suffix}_link">
-      <sensor type="ray" name="sonar${suffix}">
-        <pose>0 0 0 0 0 0</pose>
-        <visualize>true</visualize>
-        <update_rate>${update_rate}</update_rate>
-        <ray>
-          <scan>
-            <horizontal>
-              <samples>${samples}</samples>
-              <resolution>1</resolution>
-              <min_angle>-${0.5*fov}</min_angle>
-              <max_angle>${0.5*fov}</max_angle>
-            </horizontal>
-          </scan>
-          <range>
-            <min>${range_min}</min>
-            <max>${range_max}</max>
-            <resolution>0.01</resolution>
-          </range>
-          <noise>
-            <type>gaussian</type>
-            <mean>0.0</mean>
-            <stddev>${range_stddev}</stddev>
-          </noise>
-        </ray>
-        <plugin name="sonar${suffix}_controller" filename="libgazebo_ros_laser.so">
-          <topicName>${topic}</topicName>
-          <frameName>/sonar${suffix}_link</frameName>
-        </plugin>
-        <!-- TODO: Separate switchable sonar version in another macro -->
-        <!-- <plugin name="switchable_sonar{suffix}_ros_interface" filename="libuuv_gazebo_ros_switchable_gpu_ray_sensor.so">
-            <namespace>${namespace}</namespace>
-            <input_topic>${topic}</input_topic>
-        </plugin> -->
-      </sensor>
-    </gazebo>
+  <joint name="${namespace}_sonar${suffix}_joint" type="revolute">
+    <xacro:insert_block name="origin" />
+    <parent link="${parent_link}" />
+    <child link="sonar${suffix}_link" />
+    <limit upper="0" lower="0" effort="0" velocity="0" />
+    <axis xyz="1 0 0"/>
+  </joint>
+  <gazebo reference="sonar${suffix}_link">
+    <sensor type="ray" name="sonar${suffix}">
+      <pose>0 0 0 0 0 0</pose>
+      <visualize>true</visualize>
+      <update_rate>${update_rate}</update_rate>
+      <ray>
+        <scan>
+          <horizontal>
+            <samples>${samples}</samples>
+            <resolution>1</resolution>
+            <min_angle>-${0.5*fov}</min_angle>
+            <max_angle>${0.5*fov}</max_angle>
+          </horizontal>
+        </scan>
+        <range>
+          <min>${range_min}</min>
+          <max>${range_max}</max>
+          <resolution>0.01</resolution>
+        </range>
+        <noise>
+          <type>gaussian</type>
+          <mean>0.0</mean>
+          <stddev>${range_stddev}</stddev>
+        </noise>
+      </ray>
+      <plugin name="sonar${suffix}_controller" filename="libgazebo_ros_laser.so">
+        <topicName>${topic}</topicName>
+        <frameName>/sonar${suffix}_link</frameName>
+      </plugin>
+      <!-- TODO: Separate switchable sonar version in another macro -->
+      <!-- <plugin name="switchable_sonar{suffix}_ros_interface" filename="libuuv_gazebo_ros_switchable_gpu_ray_sensor.so">
+          <namespace>${namespace}</namespace>
+          <input_topic>${topic}</input_topic>
+      </plugin> -->
+    </sensor>
+  </gazebo>
   </xacro:macro>
 </robot>
