Commit message: config

File: src/packages/tauv_config/kingfisher_sim_description/urdf/base.xacro (robot description, xacro)
@@ -10,5 +10,5 @@
 <!--    <xacro:include filename="$(find kingfisher_description)/urdf/snippets.xacro"/>-->
     <xacro:property name="namespace" value="kingfisher"/>
-    <xacro:property name="mass" value="21.2"/>
+    <xacro:property name="mass" value="21.6"/>
     <!-- Center of gravity -->
     <xacro:property name="cog" value="0 0 0"/>

File: src/packages/tauv_config/kingfisher_sim_description/urdf/gazebo.xacro (robot description, xacro)
@@ -4,5 +4,5 @@
     <xacro:property name="kingfisher_cob" value="0 0 0"/>
     <!-- Vehicle's actual volume (Gazebo cannot compute the volume out of the mesh) -->
-    <xacro:property name="kingfisher_volume" value="0.0214"/>
+    <xacro:property name="kingfisher_volume" value="0.0229"/>
     <!-- Describing the dimensions of the vehicle's bounding box -->
     <xacro:property name="kingfisher_length" value="1"/>
