Commit message: Add UMD model

File: src/packages/tauv_config/kingfisher_sim_description/urdf/sensors.xacro (robot description, xacro)
@@ -6,5 +6,5 @@
             parent_link="${namespace}/base_link"
             inertial_reference_frame="${inertial_reference_frame}">
-        <origin xyz="-0.215 0 0.189" rpy="0 0 0"/>
+        <origin xyz="-0.215 0 0.189" rpy="3.14 0 1.57"/>
     </xacro:default_dvl_macro>
     <!-- Magnetometer  -->
@@ -15,5 +15,5 @@
             parent_link="${namespace}/base_link"
             inertial_reference_frame="${inertial_reference_frame}">
-        <origin xyz="0 0 0" rpy="0 0 0"/>
+        <origin xyz="0 0 0" rpy="3.14 0 1.57"/>
     </xacro:default_imu_macro>
 <!--    <xacro:default_camera-->

Commit message: Fix up controls

File: src/packages/tauv_config/kingfisher_sim_description/urdf/sensors.xacro (robot description, xacro)
@@ -6,5 +6,5 @@
             parent_link="${namespace}/base_link"
             inertial_reference_frame="${inertial_reference_frame}">
-        <origin xyz="-0.215 0 0.189" rpy="3.14 0 1.57"/>
+        <origin xyz="-0.215 0 0.189" rpy="0 0 0"/>
     </xacro:default_dvl_macro>
     <!-- Magnetometer  -->
@@ -15,5 +15,5 @@
             parent_link="${namespace}/base_link"
             inertial_reference_frame="${inertial_reference_frame}">
-        <origin xyz="0 0 0" rpy="3.14 0 1.57"/>
+        <origin xyz="0 0 0" rpy="3.14 0 0"/>
     </xacro:default_imu_macro>
 <!--    <xacro:default_camera-->

Commit message: Simulator overhaul!
Add new models
Add boilerplate for thruster plugin

More thruster work

Add first-order thruster dynamics

Add navigation state plugin

Stub out thruster manager and add static thruster transforms

Fix redundant TF transform issue

Add TAM calculation to thruster manager

Bring up PID planner

Add velocity feedforward.

Whole lot of work to clean up

Remove old kingfisher_sim_description

Restructure kingfisher_description to match kingfisher_sim_description

Clean up a bunch of namespace stuff

Camera namespace fix

Fix teleop mission namespace issue

Fix alarm server rostopic name


Fix watchdog rostopic typo


Revert change to kingfisher_description pid_planner tau


Revert MotionUtils hot start


Revert PIDPlanner d_alpha override


Add odom message to navigation state plugin

File: src/packages/tauv_config/kingfisher_sim_description/urdf/sensors.xacro (robot description, xacro)
@@ -1,36 +1,6 @@
 <?xml version="1.0"?>
 <robot xmlns:xacro="http://www.ros.org/wiki/xacro">
-    <!-- DVL  -->
-    <xacro:default_dvl_macro
-            namespace="${namespace}"
-            parent_link="${namespace}/base_link"
-            inertial_reference_frame="${inertial_reference_frame}">
-        <origin xyz="-0.215 0 0.189" rpy="0 0 0"/>
-    </xacro:default_dvl_macro>
-    <!-- Magnetometer  -->
-    <xacro:default_magnetometer namespace="${namespace}" parent_link="${namespace}/base_link"/>
-    <!-- IMU  -->
-    <xacro:default_imu_macro
-            namespace="${namespace}"
-            parent_link="${namespace}/base_link"
-            inertial_reference_frame="${inertial_reference_frame}">
-        <origin xyz="0 0 0" rpy="3.14 0 0"/>
-    </xacro:default_imu_macro>
-<!--    <xacro:default_camera-->
-<!--            namespace="${namespace}"-->
-<!--            parent_link="${namespace}/base_link"-->
-<!--            suffix="_front_left">-->
-<!--        <origin xyz="0.5 -0.05 0.0" rpy="0 0 0"/>-->
-<!--    </xacro:default_camera>-->
-<!--    <xacro:default_camera-->
-<!--            namespace="${namespace}"-->
-<!--            parent_link="${namespace}/base_link"-->
-<!--            suffix="_front_right">-->
-<!--        <origin xyz="0.5 0.05 0.0" rpy="0 0 0"/>-->
-<!--    </xacro:default_camera>-->
-    <!-- Mount a Pose 3D sensor. -->
-    <xacro:default_pose_3d_macro
-            namespace="${namespace}"
-            parent_link="${namespace}/base_link"
-            inertial_reference_frame="${inertial_reference_frame}" />
+    <xacro:navigation_state_sensor namespace="${ns}">
+        <origin xyz="0 0 0" rpy="0 0 0"/>
+    </xacro:navigation_state_sensor>
 </robot>
