Commit message: Merge in dvl and imu plugins, implement depth plugin.

File: src/packages/tauv_config/kingfisher_sim_description/urdf/default.xacro (robot description, xacro)
@@ -3,7 +3,4 @@
     <xacro:arg name="namespace" default="ns" />
     <xacro:property name="ns" value="$(arg namespace)" />
-    <xacro:include filename="$(find tauv_sim_gazebo_plugins)/urdf/utils.xacro"/>
-    <xacro:include filename="$(find tauv_sim_gazebo_plugins)/urdf/thruster_plugin.xacro"/>
-    <xacro:include filename="$(find tauv_sim_gazebo_plugins)/urdf/navigation_state_plugin.xacro"/>
     <link name="${ns}/base_link">
         <inertial>

File: src/packages/tauv_config/kingfisher_sim_description/urdf/sensors.xacro (robot description, xacro)
@@ -1,6 +1,20 @@
 <?xml version="1.0"?>
 <robot xmlns:xacro="http://www.ros.org/wiki/xacro">
+    <xacro:include filename="$(find tauv_sim_gazebo_plugins)/urdf/utils.xacro"/>
+    <xacro:include filename="$(find tauv_sim_gazebo_plugins)/urdf/navigation_state_plugin.xacro"/>
+    <xacro:include filename="$(find tauv_sim_gazebo_plugins)/urdf/teledyne_dvl_plugin.xacro"/>
+    <xacro:include filename="$(find tauv_sim_gazebo_plugins)/urdf/xsens_imu_plugin.xacro"/>
+    <xacro:include filename="$(find tauv_sim_gazebo_plugins)/urdf/depth_plugin.xacro"/>
     <xacro:navigation_state_sensor namespace="${ns}">
         <origin xyz="0 0 0" rpy="0 0 0"/>
     </xacro:navigation_state_sensor>
+    <xacro:teledyne_dvl namespace="${ns}">
+        <origin xyz="0 0 0" rpy="0 0 0"/>
+    </xacro:teledyne_dvl>
+    <xacro:xsens_imu namespace="${ns}">
+        <origin xyz="0 0 0" rpy="0 0 0"/>
+    </xacro:xsens_imu>
+    <xacro:depth_sensor namespace="${ns}">
+        <origin xyz="0 0 0" rpy="0 0 0"/>
+    </xacro:depth_sensor>
 </robot>

File: src/packages/tauv_config/kingfisher_sim_description/urdf/thrusters.xacro (robot description, xacro)
@@ -1,4 +1,6 @@
 <?xml version="1.0"?>
 <robot xmlns:xacro="http://www.ros.org/wiki/xacro">
+    <xacro:include filename="$(find tauv_sim_gazebo_plugins)/urdf/utils.xacro"/>
+    <xacro:include filename="$(find tauv_sim_gazebo_plugins)/urdf/thruster_plugin.xacro"/>
     <!--front right-->
     <xacro:t200_thruster namespace="${ns}" thruster_id="0">

Commit message: Add 2024 models to sim

File: src/packages/tauv_config/kingfisher_sim_description/urdf/default.xacro (robot description, xacro)
@@ -23,5 +23,5 @@
             <origin xyz="-0.1 0 0" rpy="0 0 1.57"/>
             <geometry>
-                <mesh filename="$(find kingfisher_sim_description)/meshes/kingfisher.dae" scale="1 1 1" />
+                <mesh filename="$(find kingfisher_sim_description)/meshes/KingfisherCoarseNoInsides.obj" scale="1 1 1" />
             </geometry>
         </visual>

Commit message: Change constants for sim in tauv config to match reality and move faster

File: src/packages/tauv_config/kingfisher_sim_description/urdf/default.xacro (robot description, xacro)
@@ -9,5 +9,5 @@
     <link name="${ns}/base_link">
         <inertial>
-            <mass value="30"/>
+            <mass value="28"/>
             <origin xyz="0 0 0" rpy="0 0 0"/>
             <inertia
@@ -21,5 +21,5 @@
         </inertial>
         <visual>
-            <origin xyz="-0.1 0 0" rpy="0 0 1.57"/>
+            <origin xyz="-0.1 0 0" rpy="0 0 3.14"/>
             <geometry>
                 <mesh filename="$(find kingfisher_sim_description)/meshes/KingfisherCoarseNoInsides.obj" scale="1 1 1" />

Commit message: push for ronnie

File: src/packages/tauv_config/kingfisher_sim_description/urdf/default.xacro (robot description, xacro)
@@ -9,5 +9,5 @@
     <link name="${ns}/base_link">
         <inertial>
-            <mass value="30"/>
+            <mass value="28"/>
             <origin xyz="0 0 0" rpy="0 0 0"/>
             <inertia
@@ -21,5 +21,5 @@
         </inertial>
         <visual>
-            <origin xyz="-0.1 0 0" rpy="0 0 1.57"/>
+            <origin xyz="-0.1 0 0" rpy="0 0 3.141592"/>
             <geometry>
                 <mesh filename="$(find kingfisher_sim_description)/meshes/KingfisherCoarseNoInsides.obj" scale="1 1 1" />

Commit message: Create simple semis 1 mission

File: src/packages/tauv_config/kingfisher_sim_description/urdf/default.xacro (robot description, xacro)
@@ -21,5 +21,5 @@
         </inertial>
         <visual>
-            <origin xyz="-0.1 0 0" rpy="0 0 3.141592"/>
+            <origin xyz="0 0 0" rpy="0 0 3.141592"/>
             <geometry>
                 <mesh filename="$(find kingfisher_sim_description)/meshes/KingfisherCoarseNoInsides.obj" scale="1 1 1" />

Commit message: reliable dead reckoning; gate - octagon - buoy (original good coordinates)

File: src/packages/tauv_config/kingfisher_sim_description/urdf/default.xacro (robot description, xacro)
@@ -21,5 +21,5 @@
         </inertial>
         <visual>
-            <origin xyz="0 0 0" rpy="0 0 3.141592"/>
+            <origin xyz="-0.1 0 0" rpy="0 0 3.141592"/>
             <geometry>
                 <mesh filename="$(find kingfisher_sim_description)/meshes/KingfisherCoarseNoInsides.obj" scale="1 1 1" />
