Commit message: Theo/missions (#155)
* Cleanup

* WIP

* Get the mission manager running

* Add mission lookup by name

* Add lock debug logs

* Add more log debugs

* Add albatross to sim

* Fix stuff

* Add Transdec model

* Add transdec models

* Implement MapClient

* Implement TransformClient

* WIP

* Implement constant acceleration trajectory

* Finish implementation of MotionClient

* Get MotionClient running with test mission

* Implement adaptive color thresholding

* Implement circle pose estimation

* Implement path marker detection

* Implement chevron detection

* Implement lid detection

* Add configurable detectors per camera

* Map visualizer

File: src/packages/tauv_config/kingfisher_sim_description/urdf/cameras.xacro (robot description, xacro)
@@ -30,5 +30,6 @@
     </link>
     <joint name="${ns}/front_oakd_joint" type="revolute">
-        <origin xyz="0.508 0 0.0508" rpy="0 0 0"/>
+<!--        <origin xyz="0.508 0 0.0508" rpy="0 0 0"/>-->
+        <origin xyz="0.5 0 0.0508" rpy="0 0 0"/>
         <parent link="${ns}/base_link"/>
         <child link="${ns}/front_oakd_link"/>
@@ -37,5 +38,6 @@
     </joint>
     <joint name="${ns}/bottom_oakd_joint" type="revolute">
-        <origin xyz="0.254 0 -0.127" rpy="1.57 1.57 0"/>
+<!--        <origin xyz="0.254 0 -0.127" rpy="1.57 1.57 0"/>-->
+        <origin xyz="0.254 0 -0.15" rpy="1.57 1.57 0"/>
         <parent link="${ns}/base_link"/>
         <child link="${ns}/bottom_oakd_link"/>

File: src/packages/tauv_config/kingfisher_sim_description/urdf/default.xacro (robot description, xacro)
@@ -20,5 +20,5 @@
         </inertial>
         <visual>
-            <origin xyz="0 0 0" rpy="0 0 0"/>
+            <origin xyz="-0.1 0 0" rpy="0 0 1.57"/>
             <geometry>
                 <mesh filename="$(find kingfisher_sim_description)/meshes/kingfisher.dae" scale="1 1 1" />
@@ -26,5 +26,5 @@
         </visual>
         <collision>
-            <origin xyz="-0.01 0 -0.08" rpy="0 0 0"/>
+            <origin xyz="-0.1 0 -0.08" rpy="0 0 0"/>
             <geometry>
                 <box size="0.986 0.538 0.366"/>

File: src/packages/tauv_config/kingfisher_sim_description/urdf/thrusters.xacro (robot description, xacro)
@@ -19,17 +19,17 @@
     <!--front right vertical-->
     <xacro:t200_thruster namespace="${ns}" thruster_id="4">
-        <origin xyz="0.23876 -0.213083 0.01115" rpy="1.5707963267949 1.5707963267949 0"/>
+        <origin xyz="0.23876 -0.213083 -0.01115" rpy="1.5707963267949 1.5707963267949 0"/>
     </xacro:t200_thruster>
     <!--front left vertical-->
     <xacro:t200_thruster namespace="${ns}" thruster_id="5">
-        <origin xyz="0.23876 0.21308 0.01115" rpy="1.5707963267949 1.5707963267949 0"/>
+        <origin xyz="0.23876 0.21308 -0.01115" rpy="1.5707963267949 1.5707963267949 0"/>
     </xacro:t200_thruster>
     <!--back right vertical-->
     <xacro:t200_thruster namespace="${ns}" thruster_id="6">
-        <origin xyz="-0.23876 -0.213083 0.01115" rpy="1.5707963267949 1.5707963267949 0"/>
+        <origin xyz="-0.23876 -0.213083 -0.01115" rpy="1.5707963267949 1.5707963267949 0"/>
     </xacro:t200_thruster>
     <!--back left vertical-->
     <xacro:t200_thruster namespace="${ns}" thruster_id="7">
-        <origin xyz="-0.23876 0.21308 0.01115" rpy="1.5707963267949 1.5707963267949 0"/>
+        <origin xyz="-0.23876 0.21308 -0.01115" rpy="1.5707963267949 1.5707963267949 0"/>
     </xacro:t200_thruster>
 </robot>

Commit message: Fix camera pose for bottom oakd

File: src/packages/tauv_config/kingfisher_sim_description/urdf/cameras.xacro (robot description, xacro)
@@ -39,5 +39,5 @@
     <joint name="${ns}/bottom_oakd_joint" type="revolute">
 <!--        <origin xyz="0.254 0 -0.127" rpy="1.57 1.57 0"/>-->
-        <origin xyz="0.254 0 -0.15" rpy="1.57 1.57 0"/>
+        <origin xyz="0.5 0 0.11" rpy="1.57 1.57 0"/>
         <parent link="${ns}/base_link"/>
         <child link="${ns}/bottom_oakd_link"/>
