Commit message: More thruster work

File: src/packages/tauv_config/new_kingfisher_sim_description/urdf/cameras.xacro (robot description, xacro)
@@ -1,71 +1,4 @@
 <?xml version="1.0"?>
-<robot name="kingfisher_sim" xmlns:xacro="http://www.ros.org/wiki/xacro">
-    <xacro:include filename="$(find tauv_sim_gazebo_plugins)/urdf/thruster_plugin.xacro"/>
-    <link name="kingfisher/base_link">
-        <inertial>
-            <mass value="30"/>
-            <origin xyz="0 0 0" rpy="0 0 0"/>
-            <inertia
-                    ixx="0.5"
-                    ixy="0.5"
-                    ixz="0.5"
-                    iyy="0.3"
-                    iyz="0.3"
-                    izz="0.5"
-            />
-        </inertial>
-        <visual>
-            <origin xyz="0 0 0" rpy="0 0 0"/>
-            <geometry>
-                <mesh filename="$(find new_kingfisher_sim_description)/meshes/kingfisher.dae" scale="1 1 1" />
-            </geometry>
-        </visual>
-        <collision>
-            <origin xyz="0 0 0" rpy="0 0 0"/>
-            <geometry>
-                <box size="1 1 1"/>
-            </geometry>
-        </collision>
-    </link>
-    <gazebo reference="kingfisher/base_link">
-        <selfCollide>false</selfCollide>
-    </gazebo>
-    <gazebo>
-        <plugin name="uuv_plugin" filename="libuuv_underwater_object_ros_plugin.so">
-            <fluid_density>1028.0</fluid_density>
-            <flow_velocity_topic>hydrodynamics/current_velocity</flow_velocity_topic>
-            <debug>true</debug>
-            <link name="kingfisher/base_link">
-                <neutrally_buoyant>0</neutrally_buoyant>
-                <volume>0.03</volume>
-                <box>
-                    <width>1</width>
-                    <length>1</length>
-                    <height>1</height>
-                </box>
-                <center_of_buoyancy>0 0 0</center_of_buoyancy>
-                <hydrodynamic_model>
-                    <type>fossen</type>
-                    <added_mass>
-                        10.7727 0 0 0 0 0
-                        0 10.7727 0 0 0 0
-                        0 0 49.7679 0 0 0
-                        0 0 0 1.0092 0 0
-                        0 0 0 0 1.0092 0
-                        0  0  0  0  0  1.0092
-                    </added_mass>
-                    <linear_damping>
-                        -9.5909 -9.5909 -42.5798 -13.3040 -13.2181 -13.3040
-                    </linear_damping>
-                    <quadratic_damping>
-                        -5.1386 -5.1386 -26.1105 0 0 0
-                    </quadratic_damping>
-                </hydrodynamic_model>
-            </link>
-        </plugin>
-    </gazebo>
-    <xacro:t200_thruster namespace="kingfisher" thruster_id="0">
-        <origin xyz="0 0 0" rpy="0 0 0"/>
-    </xacro:t200_thruster>
+<robot xmlns:xacro="http://www.ros.org/wiki/xacro">
     <xacro:property name="k1l" value="-0.389021"/>
     <xacro:property name="k2l" value="0.118184"/>
@@ -79,33 +12,11 @@
     <xacro:property name="k3r" value="0.000000"/>
     <xacro:property name="hfov" value="1.3844"/>
-    <xacro:macro name="no_visual">
-        <visual>
-            <origin xyz="0 0 0" rpy="0 ${0.5*pi} 0"/>
-            <geometry>
-                <cylinder length="${0.000001}" radius="${0.000001}" />
-            </geometry>
-        </visual>
-    </xacro:macro>
-    <xacro:macro name="no_collision">
-        <collision>
-            <origin xyz="0 0 0" rpy="0 ${0.5*pi} 0"/>
-            <geometry>
-                <cylinder length="${0.000001}" radius="${0.000001}" />
-            </geometry>
-        </collision>
-    </xacro:macro>
-   <link name="kingfisher/front_camera_left_link">
-      <inertial>
-          <mass value="0.01" />
-          <inertia ixx="0" ixy="0" ixz="0" iyy="0" iyz="0" izz="0"/>
-      </inertial>
-       <xacro:no_visual/>
-       <xacro:no_collision/>
-   </link>
+    <link name="kingfisher/front_camera_left_link">
+        <xacro:no_inertial/>
+        <xacro:no_visual/>
+        <xacro:no_collision/>
+    </link>
     <link name="kingfisher/front_camera_right_link">
-        <inertial>
-            <mass value="0.01" />
-            <inertia ixx="0" ixy="0" ixz="0" iyy="0" iyz="0" izz="0"/>
-        </inertial>
+        <xacro:no_inertial/>
         <xacro:no_visual/>
         <xacro:no_collision/>

File: src/packages/tauv_sim_gazebo_plugins/urdf/thruster_plugin.xacro (robot description, xacro)
@@ -12,28 +12,7 @@
       </joint>
       <link name="${namespace}/thruster_${thruster_id}">
-         <inertial>
-            <mass value="0.001"/>
-            <origin xyz="0 0 0" rpy="0 0 0"/>
-            <inertia
-                    ixx="0"
-                    ixy="0"
-                    ixz="0"
-                    iyy="0"
-                    iyz="0"
-                    izz="0"
-            />
-         </inertial>
-         <visual>
-            <origin xyz="0 0 0" rpy="0 ${0.5*pi} 0"/>
-            <geometry>
-               <cylinder length="${0.000001}" radius="${0.000001}" />
-            </geometry>
-         </visual>
-         <collision>
-            <origin xyz="0 0 0" rpy="0 ${0.5*pi} 0"/>
-            <geometry>
-               <cylinder length="${0.000001}" radius="${0.000001}" />
-            </geometry>
-         </collision>
+         <xacro:no_inertial/>
+         <xacro:no_visual/>
+         <xacro:no_collision/>
       </link>
       <gazebo>

Commit message: can't figure out why links don't show up for dvl/imu

File: src/packages/tauv_config/new_kingfisher_sim_description/urdf/cameras.xacro (robot description, xacro)
@@ -1,79 +1,4 @@
 <?xml version="1.0"?>
-<<<<<<< HEAD:src/packages/tauv_config/new_kingfisher_sim_description/robots/default.xacro
-<robot name="kingfisher_sim" xmlns:xacro="http://www.ros.org/wiki/xacro">
-    <xacro:include filename="$(find tauv_sim_gazebo_plugins)/urdf/thruster_plugin.xacro"/>
-    <xacro:include filename="$(find tauv_sim_gazebo_plugins)/urdf/dvl_plugin.xacro"/>
-    <link name="kingfisher/base_link">
-        <inertial>
-            <mass value="30"/>
-            <origin xyz="0 0 0" rpy="0 0 0"/>
-            <inertia
-                    ixx="0.5"
-                    ixy="0.5"
-                    ixz="0.5"
-                    iyy="0.3"
-                    iyz="0.3"
-                    izz="0.5"
-            />
-        </inertial>
-        <visual>
-            <origin xyz="0 0 0" rpy="0 0 0"/>
-            <geometry>
-                <mesh filename="$(find new_kingfisher_sim_description)/meshes/kingfisher.dae" scale="1 1 1" />
-            </geometry>
-        </visual>
-        <collision>
-            <origin xyz="0 0 0" rpy="0 0 0"/>
-            <geometry>
-                <box size="1 1 1"/>
-            </geometry>
-        </collision>
-    </link>
-    <gazebo reference="kingfisher/base_link">
-        <selfCollide>false</selfCollide>
-    </gazebo>
-    <gazebo>
-        <plugin name="uuv_plugin" filename="libuuv_underwater_object_ros_plugin.so">
-            <fluid_density>1028.0</fluid_density>
-            <flow_velocity_topic>hydrodynamics/current_velocity</flow_velocity_topic>
-            <debug>true</debug>
-            <link name="kingfisher/base_link">
-                <neutrally_buoyant>0</neutrally_buoyant>
-                <volume>0.03</volume>
-                <box>
-                    <width>1</width>
-                    <length>1</length>
-                    <height>1</height>
-                </box>
-                <center_of_buoyancy>0 0 0</center_of_buoyancy>
-                <hydrodynamic_model>
-                    <type>fossen</type>
-                    <added_mass>
-                        10.7727 0 0 0 0 0
-                        0 10.7727 0 0 0 0
-                        0 0 49.7679 0 0 0
-                        0 0 0 1.0092 0 0
-                        0 0 0 0 1.0092 0
-                        0  0  0  0  0  1.0092
-                    </added_mass>
-                    <linear_damping>
-                        -9.5909 -9.5909 -42.5798 -13.3040 -13.2181 -13.3040
-                    </linear_damping>
-                    <quadratic_damping>
-                        -5.1386 -5.1386 -26.1105 0 0 0
-                    </quadratic_damping>
-                </hydrodynamic_model>
-            </link>
-        </plugin>
-    </gazebo>
-    <xacro:t200_thruster namespace="kingfisher" thruster_id="0">
-        <origin xyz="0 0 0" rpy="0 0 0"/>
-    </xacro:t200_thruster>
-    <xacro:teledyne_dvl namespace="kingfisher">
-        <origin xyz="0 0 0" rpy="0 0 0"/>
-    </xacro:teledyne_dvl>
-=======
 <robot xmlns:xacro="http://www.ros.org/wiki/xacro">
->>>>>>> 5421fadb86b0f0fee065cbf4d3307875a5917961:src/packages/tauv_config/new_kingfisher_sim_description/urdf/cameras.xacro
     <xacro:property name="k1l" value="-0.389021"/>
     <xacro:property name="k2l" value="0.118184"/>

File: src/packages/tauv_config/new_kingfisher_sim_description/urdf/default.xacro (robot description, xacro)
@@ -3,4 +3,6 @@
     <xacro:include filename="$(find tauv_sim_gazebo_plugins)/urdf/utils.xacro"/>
     <xacro:include filename="$(find tauv_sim_gazebo_plugins)/urdf/thruster_plugin.xacro"/>
+    <xacro:include filename="$(find tauv_sim_gazebo_plugins)/urdf/teledyne_dvl_plugin.xacro"/>
+    <xacro:include filename="$(find tauv_sim_gazebo_plugins)/urdf/xsens_imu_plugin.xacro"/>
     <link name="kingfisher/base_link">
         <inertial>
@@ -68,3 +70,4 @@
     <xacro:include filename="$(find new_kingfisher_sim_description)/urdf/thrusters.xacro" />
     <xacro:include filename="$(find new_kingfisher_sim_description)/urdf/cameras.xacro" />
+    <xacro:include filename="$(find new_kingfisher_sim_description)/urdf/sensors.xacro" />
 </robot>

File: src/packages/tauv_sim_gazebo_plugins/urdf/xsens_imu_plugin.xacro (robot description, xacro)
@@ -1,17 +1,17 @@
 <?xml version="1.0"?>
 <robot xmlns:xacro="http://www.ros.org/wiki/xacro">
-   <xacro:macro name="teledyne_dvl"
+   <xacro:macro name="xsens_imu"
       params="namespace
               *origin">
-      <joint name="${namespace}/teledyne_dvl_joint" type="continuous">
+      <joint name="${namespace}/xsens_imu_joint" type="continuous">
          <xacro:insert_block name="origin"/>
          <axis xyz="1 0 0"/>
          <parent link="${namespace}/base_link"/>
-         <child link="${namespace}/teledyne_dvl"/>
+         <child link="${namespace}/xsens_imu"/>
       </joint>
-      <link name="${namespace}/teledyne_dvl">
+      <link name="${namespace}/xsens_imu">
          <inertial>
             <mass value="0.001"/>
-            <origin xyz="0 0 0" rpy="0 0 0"/>
+            <origin xyz="0 0 0" rpy="$0 0 0"/>
             <inertia
                     ixx="0"
@@ -24,5 +24,5 @@
          </inertial>
          <visual>
-            <origin xyz="0 0 0" rpy="0 ${0.5*pi} 0"/>
+            <origin xyz="0 0 0" rpy="0 0 0"/>
             <geometry>
                <cylinder length="${0.000001}" radius="${0.000001}" />
@@ -30,5 +30,5 @@
          </visual>
          <collision>
-            <origin xyz="0 0 0" rpy="0 ${0.5*pi} 0"/>
+            <origin xyz="0 0 0" rpy="0 0 0"/>
             <geometry>
                <cylinder length="${0.000001}" radius="${0.000001}" />
@@ -37,10 +37,10 @@
       </link>
       <gazebo>
-         <plugin name="${namespace}_teledyne_dvl" filename="libtauv_dvl_plugin.so">
-            <linkName>${namespace}/teledyne_dvl</linkName>
-            <jointName>${namespace}/teledyne_dvl_joint</jointName>
+         <plugin name="${namespace}_xsens_imu" filename="libtauv_xsens_imu_plugin.so">
+            <linkName>${namespace}/xsens_imu</linkName>
+            <jointName>${namespace}/xsens_imu_joint</jointName>
          </plugin>
       </gazebo>
-      <gazebo reference="${namespace}/teledyne_dvl">
+      <gazebo reference="${namespace}/xsens_imu">
          <selfCollide>false</selfCollide>
       </gazebo>
