Commit message: created branch

File: src/packages/tauv_sim_gazebo_plugins/urdf/teledyne_dvl_plugin.xacro (robot description, xacro)
@@ -1,48 +1,27 @@
 <?xml version="1.0"?>
 <robot xmlns:xacro="http://www.ros.org/wiki/xacro">
-   <xacro:macro name="teledyne_dvl"
-      params="namespace
-              *origin">
-      <joint name="${namespace}/teledyne_dvl_joint" type="continuous">
-         <xacro:insert_block name="origin"/>
-         <axis xyz="1 0 0"/>
-         <parent link="${namespace}/base_link"/>
-         <child link="${namespace}/teledyne_dvl"/>
-      </joint>
-      <link name="${namespace}/teledyne_dvl">
-         <inertial>
-            <mass value="0.001"/>
-            <origin xyz="0 0 0" rpy="$0 {0.5*pi} 0"/>
-            <inertia
-                    ixx="0"
-                    ixy="0"
-                    ixz="0"
-                    iyy="0"
-                    iyz="0"
-                    izz="0"
-            />
-         </inertial>
-         <visual>
-            <origin xyz="0 0 0" rpy="0 ${0.5*pi} 0"/>
-            <geometry>
-               <cylinder length="${0.000001}" radius="${0.000001}" />
-            </geometry>
-         </visual>
-         <collision>
-            <origin xyz="0 0 0" rpy="0 ${0.5*pi} 0"/>
-            <geometry>
-               <cylinder length="${0.000001}" radius="${0.000001}" />
-            </geometry>
-         </collision>
-      </link>
-      <gazebo>
-         <plugin name="${namespace}_teledyne_dvl" filename="libtauv_teledyne_dvl_plugin.so">
-            <linkName>${namespace}/teledyne_dvl</linkName>
-            <jointName>${namespace}/teledyne_dvl_joint</jointName>
-         </plugin>
-      </gazebo>
-      <gazebo reference="${namespace}/teledyne_dvl">
-         <selfCollide>false</selfCollide>
-      </gazebo>
-   </xacro:macro>
+    <xacro:macro name="teledyne_dvl"
+        params="namespace *origin">
+        <joint name="${namespace}/teledyne_dvl_joint" type="revolute">
+            <xacro:insert_block name="origin"/>
+            <parent link="${namespace}/base_link"/>
+            <child link="${namespace}/teledyne_dvl"/>
+            <limit upper="0" lower="0" effort="0" velocity="0"/>
+            <axis xyz="1 0 0"/>
+        </joint>
+        <link name="${namespace}/teledyne_dvl">
+            <xacro:no_inertial/>
+            <xacro:no_visual/>
+            <xacro:no_collision/>
+        </link>
+        <gazebo>
+            <plugin name="${namespace}_teledyne_dvl" filename="libtauv_teledyne_dvl_plugin.so">
+                <linkName>${namespace}/teledyne_dvl</linkName>
+                <nodeName>${namespace}_teledyne_dvl_plugin</nodeName>
+            </plugin>
+        </gazebo>
+        <gazebo reference="${namespace}/teledyne_dvl">
+            <selfCollide>false</selfCollide>
+        </gazebo>
+    </xacro:macro>
 </robot>

File: src/packages/tauv_sim_gazebo_plugins/urdf/xsens_imu_plugin.xacro (robot description, xacro)
@@ -1,48 +1,27 @@
 <?xml version="1.0"?>
 <robot xmlns:xacro="http://www.ros.org/wiki/xacro">
-   <xacro:macro name="xsens_imu"
-      params="namespace
-              *origin">
-      <joint name="${namespace}/xsens_imu_joint" type="continuous">
-         <xacro:insert_block name="origin"/>
-         <axis xyz="1 0 0"/>
-         <parent link="${namespace}/base_link"/>
-         <child link="${namespace}/xsens_imu"/>
-      </joint>
-      <link name="${namespace}/xsens_imu">
-         <inertial>
-            <mass value="0.001"/>
-            <origin xyz="0 0 0" rpy="$0 0 0"/>
-            <inertia
-                    ixx="0"
-                    ixy="0"
-                    ixz="0"
-                    iyy="0"
-                    iyz="0"
-                    izz="0"
-            />
-         </inertial>
-         <visual>
-            <origin xyz="0 0 0" rpy="0 0 0"/>
-            <geometry>
-               <cylinder length="${0.000001}" radius="${0.000001}" />
-            </geometry>
-         </visual>
-         <collision>
-            <origin xyz="0 0 0" rpy="0 0 0"/>
-            <geometry>
-               <cylinder length="${0.000001}" radius="${0.000001}" />
-            </geometry>
-         </collision>
-      </link>
-      <gazebo>
-         <plugin name="${namespace}_xsens_imu" filename="libtauv_xsens_imu_plugin.so">
-            <linkName>${namespace}/xsens_imu</linkName>
-            <jointName>${namespace}/xsens_imu_joint</jointName>
-         </plugin>
-      </gazebo>
-      <gazebo reference="${namespace}/xsens_imu">
-         <selfCollide>false</selfCollide>
-      </gazebo>
-   </xacro:macro>
+    <xacro:macro name="xsens_imu"
+        params="namespace *origin">
+        <joint name="${namespace}/xsens_imu_joint" type="revolute">
+            <xacro:insert_block name="origin"/>
+            <parent link="${namespace}/base_link"/>
+            <child link="${namespace}/xsens_imu"/>
+            <limit upper="0" lower="0" effort="0" velocity="0"/>
+            <axis xyz="1 0 0"/>
+        </joint>
+        <link name="${namespace}/xsens_imu">
+            <xacro:no_inertial/>
+            <xacro:no_visual/>
+            <xacro:no_collision/>
+        </link>
+        <gazebo>
+            <plugin name="${namespace}_xsens_imu" filename="libtauv_xsens_imu_plugin.so">
+                <linkName>${namespace}/xsens_imu</linkName>
+                <nodeName>${namespace}_xsens_imu_plugin</nodeName>
+            </plugin>
+        </gazebo>
+        <gazebo reference="${namespace}/xsens_imu">
+            <selfCollide>false</selfCollide>
+        </gazebo>
+    </xacro:macro>
 </robot>
