Commit message: fix importer, make it copy to tauv_config, check-in the urdf

File: ros_ws/src/tauv_sim/data/osprey/robot.urdf (robot description, URDF)
Before this commit: robot osprey, 24 links, 23 joints
Links:
- removed link os/body
- added link os_hull, mass 27.6559; collision mesh filename=package://assets/os_arm_base.stl; collision mesh filename=package://assets/os_dropper.stl
Joints:
- joint os/arm/base: parent os/body -> os_hull
- joint os/camera/left_frame: parent os/body -> os_hull
- joint os/camera/right_frame: parent os/body -> os_hull
- joint os/depth_frame: parent os/body -> os_hull
- joint os/dropper/left_frame: parent os/body -> os_hull
- joint os/dropper/right_frame: parent os/body -> os_hull
- joint os/dvl_frame: parent os/body -> os_hull
- joint os/imu_frame: parent os/body -> os_hull
- joint os/launcher/left/back_frame: parent os/body -> os_hull
- joint os/launcher/left/front_frame: parent os/body -> os_hull
- joint os/launcher/right/back_frame: parent os/body -> os_hull
- joint os/launcher/right/front_frame: parent os/body -> os_hull
- joint os/thruster/alh_frame: parent os/body -> os_hull
- joint os/thruster/alv_frame: parent os/body -> os_hull
- joint os/thruster/arh_frame: parent os/body -> os_hull
- joint os/thruster/arv_frame: parent os/body -> os_hull
- joint os/thruster/flh_frame: parent os/body -> os_hull
- joint os/thruster/flv_frame: parent os/body -> os_hull
- joint os/thruster/frh_frame: parent os/body -> os_hull
- joint os/thruster/frv_frame: parent os/body -> os_hull
