Commit message: hella stuff

File: ros_ws/src/tauv_config/urdf/osprey.urdf (robot description, URDF)
Before this commit: robot osprey, 12 links, 11 joints
Links:
- removed link base_link
- removed link depth
- removed link dvl
- removed link imu
- removed link thruster/hlb
- removed link thruster/hlf
- removed link thruster/hrb
- removed link thruster/hrf
- removed link thruster/vlb
- removed link thruster/vlf
- removed link thruster/vrb
- removed link thruster/vrf
- added link os/arm/intake, mass 1e-9
- added link os/arm/thruster, mass 1e-9
- added link os/body, mass 20.4159; collision mesh filename=package://assets/frame.stl; collision mesh filename=package://assets/os/body.stl
- added link os/camera/left, mass 1e-9
- added link os/camera/right, mass 1e-9
- added link os/depth, mass 1e-9
- added link os/dropper/left, mass 1e-9
- added link os/dropper/right, mass 1e-9
- added link os/dvl, mass 1e-9
- added link os/launcher/left/front, mass 1e-9
- added link os/launcher/right/back, mass 1e-9
- added link os/launcher/right/front, mass 1e-9
- added link os/thruster/alh, mass 1e-9
- added link os/thruster/alv, mass 1e-9
- added link os/thruster/arh, mass 1e-9
- added link os/thruster/arv, mass 1e-9
- added link os/thruster/flh, mass 1e-9
- added link os/thruster/flv, mass 1e-9
- added link os/thruster/frh, mass 1e-9
- added link os/thruster/frv, mass 1e-9
- added link os_arm_link, mass 0.682725; collision mesh filename=package://assets/os_arm_link.stl; visual mesh filename=package://assets/os_arm_link.stl
- added link os_arm_tube, mass 0.780591; collision mesh filename=package://assets/os_arm_tube.stl; visual mesh filename=package://assets/os_arm_tube.stl
Joints:
- removed joint base_to_depth
- removed joint base_to_dvl
- removed joint base_to_hlb
- removed joint base_to_hlf
- removed joint base_to_hrb
- removed joint base_to_hrf
- removed joint base_to_imu
- removed joint base_to_vlb
- removed joint base_to_vlf
- removed joint base_to_vrb
- removed joint base_to_vrf
- added joint os/arm/base: type revolute, parent os/body, child os_arm_link, origin xyz=0.279674 -0.0348629 0.119766 rpy=1.5708 1.79519e-16 3.14159, axis 0 0 1, limit lower=-2.79253 upper=8.88178e-16 effort=10 velocity=10
- added joint os/arm/intake_frame: type fixed, parent os_arm_tube, child os/arm/intake, origin xyz=1.66533e-16 -0.1397 -0.0587375 rpy=1.5708 -1.5708 0, axis 0 0 0
- added joint os/arm/link: type revolute, parent os_arm_link, child os_arm_tube, origin xyz=-0.204288 0.0743547 0.02185 rpy=-3.14159 -1.67456e-16 -1.62897e-16, axis 0 0 1, limit lower=-3.141592653589793 upper=3.141592653589793 effort=10 velocity=10, mimic joint=os/arm/base multiplier=-0.6666666666666666
- added joint os/arm/thruster_frame: type fixed, parent os_arm_tube, child os/arm/thruster, origin xyz=0.001 0.031518 -0.0587375 rpy=1.5708 -1.5708 0, axis 0 0 0
- added joint os/camera/left_frame: type fixed, parent os/body, child os/camera/left, origin xyz=0.300784 -0.10975 0.192154 rpy=1.5708 2.89093e-31 1.5708, axis 0 0 0
- added joint os/camera/right_frame: type fixed, parent os/body, child os/camera/right, origin xyz=0.300784 0.20775 0.192154 rpy=1.5708 -2.29489e-31 1.5708, axis 0 0 0
- added joint os/depth_frame: type fixed, parent os/body, child os/depth, origin xyz=0.240087 0.0871 -0.0554465 rpy=-1.5708 -2.33274e-31 -1.5708, axis 0 0 0
- added joint os/dropper/left_frame: type fixed, parent os/body, child os/dropper/left, origin xyz=-0.181328 0.173632 0.118106 rpy=-7.00728e-16 -8.04509e-16 -1.5708, axis 0 0 0
- added joint os/dropper/right_frame: type fixed, parent os/body, child os/dropper/right, origin xyz=-0.181328 0.206232 0.118106 rpy=-7.00728e-16 -8.04509e-16 -1.5708, axis 0 0 0
- added joint os/dvl_frame: type fixed, parent os/body, child os/dvl, origin xyz=-0.103308 0.0490119 0.0448185 rpy=-1.79692e-16 2.07039e-14 -1.5708, axis 0 0 0
- added joint os/launcher/left/front_frame: type fixed, parent os/body, child os/launcher/left/front, origin xyz=0.340329 0.12539 0.0589185 rpy=-1.5708 -1.93383e-14 -1.5708, axis 0 0 0
- added joint os/launcher/right/back_frame: type fixed, parent os/body, child os/launcher/right/back, origin xyz=0.121316 0.17974 0.0589185 rpy=-1.5708 -1.93383e-14 -1.5708, axis 0 0 0
- added joint os/launcher/right/front_frame: type fixed, parent os/body, child os/launcher/right/front, origin xyz=0.340329 0.17974 0.0589185 rpy=-1.5708 -1.93383e-14 -1.5708, axis 0 0 0
- added joint os/thruster/alh_frame: type fixed, parent os/body, child os/thruster/alh, origin xyz=-0.187324 -0.177973 -0.0540697 rpy=-1.5708 -3.70241e-16 -0.785398, axis 0 0 0
- added joint os/thruster/alv_frame: type fixed, parent os/body, child os/thruster/alv, origin xyz=-0.056594 -0.19685 0.0478974 rpy=-9.8687e-17 -1.5708 0, axis 0 0 0
- added joint os/thruster/arh_frame: type fixed, parent os/body, child os/thruster/arh, origin xyz=-0.187324 0.275973 -0.0540697 rpy=-1.5708 3.75523e-15 0.785398, axis 0 0 0
- added joint os/thruster/arv_frame: type fixed, parent os/body, child os/thruster/arv, origin xyz=-0.056594 0.29485 0.0478974 rpy=-1.5708 -1.5708 0, axis 0 0 0
- added joint os/thruster/flh_frame: type fixed, parent os/body, child os/thruster/flh, origin xyz=0.284088 -0.156383 -0.0540697 rpy=-1.5708 1.88842e-17 0.785398, axis 0 0 0
- added joint os/thruster/flv_frame: type fixed, parent os/body, child os/thruster/flv, origin xyz=0.131768 -0.19685 0.0478974 rpy=-9.8687e-17 -1.5708 0, axis 0 0 0
- added joint os/thruster/frh_frame: type fixed, parent os/body, child os/thruster/frh, origin xyz=0.284088 0.254383 -0.0540697 rpy=-1.5708 3.23543e-16 -0.785398, axis 0 0 0
- added joint os/thruster/frv_frame: type fixed, parent os/body, child os/thruster/frv, origin xyz=0.131768 0.29485 0.0478974 rpy=-3.14159 -1.5708 0, axis 0 0 0

Commit message: unfuck thruster frames

File: ros_ws/src/tauv_config/urdf/osprey.urdf (robot description, URDF)
Before this commit: robot osprey, 24 links, 23 joints
Links:
- added link os/hull, mass 27.6559; collision mesh filename=package://assets/os/hull.stl; collision mesh filename=package://assets/os_arm_base.stl
- link os/body: mass 27.6559 -> 1e-09; geometry collision mesh filename=package://assets/frame.stl; visual mesh filename=package://assets/frame.stl
Joints:
- added joint os/body_frame: type fixed, parent os/hull, child os/body, origin xyz=9.3735e-36 -1.53081e-19 0 rpy=0 0 3.14159, axis 0 0 1, limit effort=10 velocity=10
- joint os/arm/base: parent os/body -> os/hull
- joint os/arm/intake_frame: origin xyz=2.08167e-16 -0.1397 -0.0587375 rpy=1.5708 -1.5708 0 -> xyz=1.52656e-16 -0.1397 -0.0587375 rpy=1.5708 -1.5708 0
- joint os/camera/left_frame: parent os/body -> os/hull
- joint os/camera/right_frame: parent os/body -> os/hull
- joint os/depth_frame: parent os/body -> os/hull
- joint os/dropper/left_frame: parent os/body -> os/hull
- joint os/dropper/right_frame: parent os/body -> os/hull
- joint os/dvl_frame: parent os/body -> os/hull
- joint os/imu_frame: parent os/body -> os/hull
- joint os/launcher/left/back_frame: parent os/body -> os/hull
- joint os/launcher/left/front_frame: parent os/body -> os/hull
- joint os/launcher/right/back_frame: parent os/body -> os/hull
- joint os/launcher/right/front_frame: parent os/body -> os/hull
- joint os/thruster/alh_frame: parent os/body -> os/hull
- joint os/thruster/alv_frame: origin xyz=0.094181 0.24585 0.0230414 rpy=3.14159 -1.5708 0 -> xyz=0.094181 0.24585 0.0230414 rpy=9.8687e-17 -1.5708 0; parent os/body -> os/hull
- joint os/thruster/arh_frame: parent os/body -> os/hull
- joint os/thruster/arv_frame: origin xyz=0.094181 -0.24585 0.0230414 rpy=1.5708 -1.5708 0 -> xyz=0.094181 -0.24585 0.0230414 rpy=0 -1.5708 0; parent os/body -> os/hull
- joint os/thruster/flh_frame: parent os/body -> os/hull
- joint os/thruster/flv_frame: origin xyz=-0.094181 0.24585 0.0230414 rpy=3.14159 -1.5708 0 -> xyz=-0.094181 0.24585 0.0230414 rpy=0.0 -1.5708 0.0; parent os/body -> os/hull
- joint os/thruster/frh_frame: parent os/body -> os/hull
- joint os/thruster/frv_frame: origin xyz=-0.094181 -0.24585 0.0230414 rpy=1.10637e-15 -1.5708 0 -> xyz=-0.094181 -0.24585 0.0230414 rpy=0.0 -1.5708 0; parent os/body -> os/hull

File: ros_ws/src/tauv_sim/data/osprey/robot.urdf (robot description, URDF)
Before this commit: robot osprey, 24 links, 23 joints
Links:
- added link frame, mass 1e-09; collision mesh filename=package://assets/frame.stl; visual mesh filename=package://assets/frame.stl
Joints:
- added joint os/body: type fixed, parent os_hull, child frame, origin xyz=9.3735e-36 -1.53081e-19 0 rpy=3.14159 -0 -3.14159, axis 0 0 1, limit effort=10 velocity=10
- joint os/arm/intake_frame: origin xyz=2.08167e-16 -0.1397 -0.0587375 rpy=1.5708 -1.5708 0 -> xyz=1.52656e-16 -0.1397 -0.0587375 rpy=1.5708 -1.5708 0
- joint os/thruster/alv_frame: origin xyz=0.094181 0.24585 0.0230414 rpy=3.14159 -1.5708 0 -> xyz=0.094181 0.24585 0.0230414 rpy=9.8687e-17 1.5708 0
- joint os/thruster/arv_frame: origin xyz=0.094181 -0.24585 0.0230414 rpy=1.5708 -1.5708 0 -> xyz=0.094181 -0.24585 0.0230414 rpy=-1.5708 1.5708 0
- joint os/thruster/flv_frame: origin xyz=-0.094181 0.24585 0.0230414 rpy=3.14159 -1.5708 0 -> xyz=-0.094181 0.24585 0.0230414 rpy=9.8687e-17 1.5708 0
- joint os/thruster/frv_frame: origin xyz=-0.094181 -0.24585 0.0230414 rpy=1.10637e-15 -1.5708 0 -> xyz=-0.094181 -0.24585 0.0230414 rpy=3.14159 1.5708 0

Commit message: stuff

File: ros_ws/src/tauv_config/urdf/osprey.urdf (robot description, URDF)
Before this commit: robot osprey, 25 links, 24 joints
Joints:
- joint os/imu_frame: origin xyz=0.037587 0.049 -0.024856 rpy=2.71051e-20 -6.12323e-17 -3.14159 -> xyz=0.037587 0.049 -0.024856 rpy=2.71051e-20 -6.12323e-17 0

Commit message: all frames are broken

File: ros_ws/src/tauv_config/urdf/osprey.urdf (robot description, URDF)
Before this commit: robot osprey, 25 links, 24 joints
Joints:
- joint os/imu_frame: origin xyz=0.037587 0.049 -0.024856 rpy=2.71051e-20 -6.12323e-17 0 -> xyz=0.037587 0.049 -0.024856 rpy=3.14159 0.0 0.0
